File: supercap/supercap/supercap.kicad_pcb (KiCad board)
At the start: 4 copper layers, 70 x 174 mm, 60 parts, among them J201 Conn_01x02, J202 Conn_01x02, J203 Power Output, J204 CAN2 PLUG, Q201 100V 34A PMOS, Q202 100V 34A PMOS, Q203 100V 34A PMOS, Q204 Q_NMOS_GSD, Q205 100V 34A PMOS, Q206 100V 34A PMOS, Q207 100V 34A PMOS

Commit message: Rev 2 Supercap PCB, updates to Motherboard in progress
Parts:
- removed C201, C222: 1uF, Capacitor_SMD:C_0805_2012Metric
- removed the G*** at (-66.6, 25.3)
- removed the G*** at (-54.7, 65.7)
- removed the G*** at (-75.1, 63.7)
- removed the G*** at (-70.8, 75.1)
- removed the G*** at (-45.3, 22.8)
- removed the G*** at (-59.4, 73.0)
- removed the G*** at (-57.6, 29.4)
- removed the G*** at (-54.3, 18.8)
- removed the G*** at (-78.1, 27.3)
- removed the G*** at (-50.4, 77.1)
- removed the G*** at (-63.7, 61.6)
- removed the G*** at (-65.7, 20.8)
- removed H201, H202: MountingHole_Pad, supercap:Sinhoo-SMTSO40x-C2916378
- removed H203, H204: MountingHole, supercap:MountingHole_3.9mm_Plastite_#6
- removed J201: Conn_01x02, Connector_Anderson:PowerPole_PP45_1336G1_1x2_Horizontal
- removed J204: CAN2 PLUG, supercap:PINREX-744-81-04TW00 _1x04_P2.54mm_Vertical
- removed JP201, JP202, JP203, JP204, JP205, JP206, JP207: SolderJumper_2_Open, Jumper:SolderJumper-2_P1.3mm_Open_RoundedPad1.0x1.5mm
- removed Q203: 100V 34A PMOS, Package_TO_SOT_SMD:TO-252-2
- removed R201, R203: 10k, Resistor_SMD:R_0805_2012Metric
- removed R202, R204: 20k, Resistor_SMD:R_0805_2012Metric
- added C1: 20p, Capacitor_SMD:C_0603_1608Metric, F.Cu at (144.4, 98.6)
- added C14: 100n, Capacitor_SMD:C_0603_1608Metric, F.Cu at (151.4, 78.8)
- added C15: 100n, Capacitor_SMD:C_0603_1608Metric, F.Cu at (150.6, 93.5)
- added C16: 1u, Capacitor_SMD:C_0603_1608Metric, F.Cu at (148.3, 77.9)
- added C2: 20p, Capacitor_SMD:C_0603_1608Metric, F.Cu at (149.9, 95.7)
- added C28: 1u, Capacitor_SMD:C_0603_1608Metric, F.Cu at (88.7, 160.2)
- added C29: 100n, Capacitor_SMD:C_0603_1608Metric, F.Cu at (154.3, 79.6)
- added C3: 1u, Capacitor_SMD:C_0603_1608Metric, F.Cu at (98.5, 162.6)
- added C30: 100n, Capacitor_SMD:C_0603_1608Metric, F.Cu at (149.8, 77.9)
- added C31: 100n, Capacitor_SMD:C_0603_1608Metric, F.Cu at (154.8, 89.9)
- added C32: 1u, Capacitor_SMD:C_0603_1608Metric, F.Cu at (154.2, 81.1)
- added C33: 100n, Capacitor_SMD:C_0603_1608Metric, F.Cu at (154.8, 88.3)
- added C34: 100n, Capacitor_SMD:C_0603_1608Metric, F.Cu at (141.8, 82.2)
- added C35: 100n, Capacitor_SMD:C_0603_1608Metric, F.Cu at (149.1, 93.5)
- added C36: 100n, Capacitor_SMD:C_0603_1608Metric, F.Cu at (154.1, 82.6)
- added C37: 100n, Capacitor_SMD:C_0603_1608Metric, F.Cu at (76.3, 131.0)
- added C38: 100n, Capacitor_SMD:C_0603_1608Metric, F.Cu at (158.0, 124.1)
- added C39: 1u, Capacitor_SMD:C_0603_1608Metric, F.Cu at (112.7, 83.3)
- added C4: 100n, Capacitor_SMD:C_0603_1608Metric, F.Cu at (149.1, 75.5)
- added C40: 47uF 63V solid, Capacitor_THT:CP_Radial_D8.0mm_P3.50mm, F.Cu at (145.6, 49.9)
- added C41: 100n, Capacitor_SMD:C_0603_1608Metric, F.Cu at (114.4, 83.3)
- added C42: 22uF 25V, Capacitor_SMD:C_0805_2012Metric, F.Cu at (159.4, 33.3)
- added C43: 4.7uF 100V, Capacitor_SMD:C_1210_3225Metric, F.Cu at (141.3, 43.2)
- added C44: 100nF 100V, Capacitor_SMD:C_0805_2012Metric, F.Cu at (144.6, 43.8)
- added C45: 1u, Capacitor_SMD:C_0603_1608Metric, F.Cu at (158.9, 49.4)
- added C46: 22nF, Capacitor_SMD:C_0603_1608Metric, F.Cu at (159.6, 38.6)
- added C47: 100n, Capacitor_SMD:C_0603_1608Metric, F.Cu at (155.8, 38.9)
- added C48: 10u, Capacitor_SMD:C_0805_2012Metric, F.Cu at (162.3, 49.3)
- added C49: 22pF, Capacitor_SMD:C_0603_1608Metric, F.Cu at (162.5, 32.5)
- added C50: 47uF 10v, Capacitor_SMD:C_0805_2012Metric, F.Cu at (162.8, 37.3)
- added C51: 47pf, Capacitor_SMD:C_0603_1608Metric, F.Cu at (156.0, 44.4)
- added C52: 22uF 25V, Capacitor_SMD:C_0805_2012Metric, F.Cu at (164.9, 37.3)
- added C53: 220uF 25V, Capacitor_SMD:CP_Elec_6.3x7.7, F.Cu at (144.2, 32.0)
- added D1: B5819W SL, Diode_SMD:D_SOD-123, F.Cu at (161.6, 73.5)
- added D10: 2.4v zener, supercap:DIO_PESD5V0S1UL_315, F.Cu at (110.0, 94.9)
- added D11: 2.4v zener, supercap:DIO_PESD5V0S1UL_315, F.Cu at (110.0, 113.8)
- added D12: 2.4v zener, supercap:DIO_PESD5V0S1UL_315, F.Cu at (91.0, 113.7)
- added D13: 2.4v zener, supercap:DIO_PESD5V0S1UL_315, F.Cu at (91.0, 94.8)
- added D14: 2.4v zener, supercap:DIO_PESD5V0S1UL_315, F.Cu at (91.0, 75.6)
- added D15: 2.4v zener, supercap:DIO_PESD5V0S1UL_315, F.Cu at (91.0, 56.9)
- added D16: 2.4v zener, supercap:DIO_PESD5V0S1UL_315, F.Cu at (91.0, 37.6)
- added D17: 2.4v zener, supercap:DIO_PESD5V0S1UL_315, F.Cu at (72.0, 37.9)
- added D18: 2.4v zener, supercap:DIO_PESD5V0S1UL_315, F.Cu at (72.0, 57.0)
- added D19: 2.4v zener, supercap:DIO_PESD5V0S1UL_315, F.Cu at (72.1, 75.8)
- added D2: 2.4v zener, supercap:DIO_PESD5V0S1UL_315, F.Cu at (129.0, 113.8)
- added D20: 2.4v zener, supercap:DIO_PESD5V0S1UL_315, F.Cu at (72.0, 95.0)
- added D21: 2.4v zener, supercap:DIO_PESD5V0S1UL_315, F.Cu at (72.0, 114.2)
- added D22: SMAJ51A, Diode_SMD:D_SMA, F.Cu at (137.5, 125.2)
- added D23: D, Diode_SMD:D_SMA, F.Cu at (134.5, 46.2)
- added D24: SMAJ51A, Diode_SMD:D_SMA, F.Cu at (81.0, 154.3)
- added D25: D, Diode_SMD:D_SMA, F.Cu at (134.5, 50.3)
- added D26: SS310, Diode_SMD:D_SMA, F.Cu at (144.2, 38.6)
- added D27: 1N4148WS, Diode_SMD:D_SOD-323, F.Cu at (116.5, 86.2)
- added D28: 1N4148WS, Diode_SMD:D_SOD-323, F.Cu at (157.8, 97.7)
- added D29: 1N4148WS, Diode_SMD:D_SOD-323, F.Cu at (67.9, 154.8)
- added D3: 2.4v zener, supercap:DIO_PESD5V0S1UL_315, F.Cu at (129.0, 94.7)
- added D30: WS2812B, RP2040_minimal:LED_WS2812_3528_3.5x2.8mm_P1.5mm, F.Cu at (161.9, 113.1)
- added D31: WS2812B, RP2040_minimal:LED_WS2812_3528_3.5x2.8mm_P1.5mm, F.Cu at (161.9, 116.3)
- added D32: WS2812B, RP2040_minimal:LED_WS2812_3528_3.5x2.8mm_P1.5mm, F.Cu at (161.9, 119.6)
- added D33: Zener 10v, Diode_SMD:D_SOD-323, F.Cu at (136.9, 169.9)
- added D34: Zener 10v, Diode_SMD:D_SOD-323, F.Cu at (99.2, 124.5)
- added D4: 2.4v zener, supercap:DIO_PESD5V0S1UL_315, F.Cu at (129.0, 75.3)
- added D5: 2.4v zener, supercap:DIO_PESD5V0S1UL_315, F.Cu at (129.0, 56.6)
- added D6: 2.4v zener, supercap:DIO_PESD5V0S1UL_315, F.Cu at (129.0, 37.4)
- added D7: 2.4v zener, supercap:DIO_PESD5V0S1UL_315, F.Cu at (110.0, 37.9)
- added D8: 2.4v zener, supercap:DIO_PESD5V0S1UL_315, F.Cu at (110.0, 56.6)
- added D9: 2.4v zener, supercap:DIO_PESD5V0S1UL_315, F.Cu at (110.0, 75.8)
- added G***: LOGO, taylor_footprints:twisted_icon, F.Cu at (115.2, 66.4)
- added G***: LOGO, taylor_footprints:twisted, F.Cu at (104.2, 64.5)
- added G***: LOGO, taylor_footprints:twisted_2, F.Cu at (91.9, 68.4)
- added G***: LOGO, taylor_footprints:twisted_icon, B.Cu at (165.8, -85.5)
- added G***: LOGO, taylor_footprints:twisted_2, B.Cu at (186.3, -83.4)
- added G***: LOGO, taylor_footprints:twisted, B.Cu at (177.3, -87.5)
- added H1: MountingHole, supercap:MountingHole_3.9mm_Plastite_#6, F.Cu at (163.5, 171.5)
- added H2: MountingHole, supercap:MountingHole_3.9mm_Plastite_#6, F.Cu at (63.0, 171.5)
- added H3: MountingHole, supercap:MountingHole_3.9mm_Plastite_#6, F.Cu at (163.5, 24.5)
- added H4: MountingHole, supercap:MountingHole_3.9mm_Plastite_#6, F.Cu at (63.0, 24.5)
- added J1: CPU2 USB, Connector_USB:USB_C_Receptacle_XKB_U262-16XN-4BVC11, F.Cu at (164.5, 82.2)
- added J2: Conn_01x06, parts:Ckmtw-W-2510S06P_1x06_P2.54mm_Vertical, F.Cu at (153.8, 60.4)
- added J4: Conn_01x02, Connector_Anderson:PowerPole_PP45_1336G1_1x2_Horizontal, F.Cu at (138.7, 155.1)
- added J6: CAN2 PLUG, supercap:PINREX-744-81-04TW00 _1x04_P2.54mm_Vertical, F.Cu at (163.6, 106.3)
- added JP1: SolderJumper_2_Open, Jumper:SolderJumper-2_P1.3mm_Open_RoundedPad1.0x1.5mm, B.Cu at (132.5, 136.5)
- added JP10: SolderJumper_2_Open, Jumper:SolderJumper-2_P1.3mm_Open_RoundedPad1.0x1.5mm, B.Cu at (92.0, 153.2)
- added JP2: SolderJumper_2_Open, Jumper:SolderJumper-2_P1.3mm_Open_RoundedPad1.0x1.5mm, B.Cu at (129.9, 136.5)
- added JP3: SolderJumper_2_Open, Jumper:SolderJumper-2_P1.3mm_Open_RoundedPad1.0x1.5mm, B.Cu at (127.1, 136.5)
- added JP4: SolderJumper_2_Open, Jumper:SolderJumper-2_P1.3mm_Open_RoundedPad1.0x1.5mm, B.Cu at (124.3, 136.5)
- added JP5: SolderJumper_2_Open, Jumper:SolderJumper-2_P1.3mm_Open_RoundedPad1.0x1.5mm, B.Cu at (121.5, 136.5)
- added JP6: SolderJumper_2_Open, Jumper:SolderJumper-2_P1.3mm_Open_RoundedPad1.0x1.5mm, B.Cu at (92.0, 143.0)
- added JP7: SolderJumper_2_Open, Jumper:SolderJumper-2_P1.3mm_Open_RoundedPad1.0x1.5mm, B.Cu at (92.0, 145.6)
- added JP8: SolderJumper_2_Open, Jumper:SolderJumper-2_P1.3mm_Open_RoundedPad1.0x1.5mm, B.Cu at (92.0, 148.1)
- added JP9: SolderJumper_2_Open, Jumper:SolderJumper-2_P1.3mm_Open_RoundedPad1.0x1.5mm, B.Cu at (92.0, 150.7)
- added L1: 10uH, Inductor_SMD:L_Sunlord_SWPA5040S, F.Cu at (160.6, 42.2)
- added L2: 47uH, Inductor_SMD:L_Chilisin_BMRB00060612, F.Cu at (151.4, 35.9)
- added Q1: Q_NMOS_GSD, Package_TO_SOT_SMD:SOT-23, F.Cu at (129.9, 166.1)
- added Q10: Q_NMOS_GSD, Package_TO_SOT_SMD:SOT-23, F.Cu at (155.1, 110.1)
- added Q12: 100V 34A PMOS, Package_TO_SOT_SMD:TO-252-2, F.Cu at (94.7, 154.6)
- added Q2: 100V 34A PMOS, Package_TO_SOT_SMD:TO-252-2, F.Cu at (129.3, 137.0)
- added Q3: 100V 34A PMOS, Package_TO_SOT_SMD:TO-252-2, F.Cu at (129.3, 160.9)
- added Q6: 100V 34A PMOS, Package_TO_SOT_SMD:TO-252-2, F.Cu at (119.5, 137.0)
- added Q7: 100V 34A PMOS, Package_TO_SOT_SMD:TO-252-2, F.Cu at (119.6, 160.9)
- added Q8: 100V 34A PMOS, Package_TO_SOT_SMD:TO-252-2, F.Cu at (119.5, 144.3)
- added Q9: 100V 34A PMOS, Package_TO_SOT_SMD:TO-252-2, F.Cu at (119.6, 153.5)
- added R1: 10k, Resistor_SMD:R_1206_3216Metric, F.Cu at (134.4, 166.0)
- added R10: 10k, Resistor_SMD:R_0603_1608Metric, F.Cu at (86.2, 157.3)
- added R11: 27, Resistor_SMD:R_0603_1608Metric, F.Cu at (158.9, 78.6)
- added R12: 27, Resistor_SMD:R_0603_1608Metric, F.Cu at (157.4, 78.6)
- added R13: 3mΩ, Resistor_SMD:R_2512_6332Metric, F.Cu at (87.4, 131.1)
- added R14: 3mΩ, Resistor_SMD:R_2512_6332Metric, F.Cu at (147.9, 127.4)
- added R15: 3mΩ, Resistor_SMD:R_2512_6332Metric, F.Cu at (83.2, 131.1)
- added R16: 100R 2W, Resistor_SMD:R_2512_6332Metric, F.Cu at (138.1, 106.2)
- added R17: 100R 2W, Resistor_SMD:R_2512_6332Metric, F.Cu at (138.1, 114.3)
- added R18: 100R 2W, Resistor_SMD:R_2512_6332Metric, F.Cu at (142.3, 106.2)
- added R19: 100R 2W, Resistor_SMD:R_2512_6332Metric, F.Cu at (142.2, 114.3)
- added R2: 1k 2 watt, Resistor_SMD:R_2512_6332Metric, F.Cu at (128.2, 128.2)
- added R20: 100R 2W, Resistor_SMD:R_2512_6332Metric, F.Cu at (146.4, 106.2)
- added R21: 100R 2W, Resistor_SMD:R_2512_6332Metric, F.Cu at (146.4, 114.3)
- added R22: 100R 2W, Resistor_SMD:R_2512_6332Metric, F.Cu at (150.9, 106.2)
- added R23: 100R 2W, Resistor_SMD:R_2512_6332Metric, F.Cu at (150.9, 114.2)
- added R24: 10k, Resistor_SMD:R_1206_3216Metric, F.Cu at (99.4, 126.8)
- added R25: 50mΩ, Resistor_SMD:R_0603_1608Metric, F.Cu at (144.5, 41.3)
- added R26: 10Ω, Resistor_SMD:R_0603_1608Metric, F.Cu at (155.0, 41.2)
- added R27: 50k 0.1%, Resistor_SMD:R_0603_1608Metric, F.Cu at (113.5, 88.0)
- added R28: 50k 0.1%, Resistor_SMD:R_0603_1608Metric, F.Cu at (116.8, 88.0)
- added R29: 5.1k 0.1%, Resistor_SMD:R_0603_1608Metric, F.Cu at (120.1, 88.0)
- added R3: 1k 2 watt, Resistor_SMD:R_2512_6332Metric, F.Cu at (132.3, 128.2)
- added R30: 110k 0.1%, Resistor_SMD:R_0603_1608Metric, F.Cu at (164.2, 32.5)
- added R31: 15k 0.1%, Resistor_SMD:R_0603_1608Metric, F.Cu at (163.4, 34.8)
- added R32: 300k, Resistor_SMD:R_0603_1608Metric, F.Cu at (154.3, 44.4)
- added R33: 21.5k, Resistor_SMD:R_0603_1608Metric, F.Cu at (150.2, 46.7)
- added R34: 50k 0.1%, Resistor_SMD:R_0603_1608Metric, F.Cu at (157.2, 103.1)
- added R35: 50k 0.1%, Resistor_SMD:R_0603_1608Metric, F.Cu at (156.7, 100.6)
- added R36: 5.1k 0.1%, Resistor_SMD:R_0603_1608Metric, F.Cu at (158.7, 100.6)
- added R37: 50k 0.1%, Resistor_SMD:R_0603_1608Metric, F.Cu at (67.8, 160.2)
- added R38: 50k 0.1%, Resistor_SMD:R_0603_1608Metric, F.Cu at (66.8, 157.6)
- added R39: 5.1k 0.1%, Resistor_SMD:R_0603_1608Metric, F.Cu at (68.8, 157.6)
- added R4: 1.1k, Resistor_SMD:R_0603_1608Metric, F.Cu at (146.4, 68.3)
- added R40: 2k 2 watt, Resistor_SMD:R_2512_6332Metric, F.Cu at (131.3, 170.3)
- added R41: 2k 2 watt, Resistor_SMD:R_2512_6332Metric, F.Cu at (99.9, 121.4)
- added R42: 120R, Resistor_SMD:R_0603_1608Metric, F.Cu at (164.1, 94.8)
- added R43: 5.1k, Resistor_SMD:R_0603_1608Metric, F.Cu at (153.4, 96.3)
- added R5: DNS, Resistor_SMD:R_0402_1005Metric, F.Cu at (141.4, 79.8)
- added R6: 5.1k, Resistor_SMD:R_0603_1608Metric, F.Cu at (158.8, 85.8)
- added R7: 5.1k, Resistor_SMD:R_0603_1608Metric, F.Cu at (161.8, 76.0)
- added R8: 1.1k, Resistor_SMD:R_0603_1608Metric, F.Cu at (147.6, 93.9)
- added R9: 10k, Resistor_SMD:R_0603_1608Metric, F.Cu at (95.3, 159.9)
- added SW1: SW_MEC_5G, supercap:SW_TS_1101_C_W, F.Cu at (161.5, 65.3)
- added SW2: SW_MEC_5G, supercap:SW_TS_1101_C_W, F.Cu at (136.0, 81.4)
- added SW3: SW_MEC_5G, supercap:SW_TS_1101_C_W, F.Cu at (136.0, 69.4)
- added SW4: SW_MEC_5G, supercap:SW_TS_1101_C_W, F.Cu at (136.0, 93.4)
- added TH1: Thermistor 10k, Resistor_SMD:R_0603_1608Metric, F.Cu at (125.1, 148.9)
- added TH2: Thermistor 10k, Resistor_SMD:R_0603_1608Metric, F.Cu at (88.2, 153.2)
- added TP1: TestPoint, TestPoint:TestPoint_Loop_D2.60mm_Drill1.6mm_Beaded, F.Cu at (155.9, 70.2)
- added TP2: TestPoint, TestPoint:TestPoint_Pad_D2.0mm, B.Cu at (163.4, 84.1)
- added TP3: TestPoint, TestPoint:TestPoint_Pad_D2.0mm, B.Cu at (163.5, 80.1)
- added TP4: TestPoint, TestPoint:TestPoint_Pad_D2.0mm, B.Cu at (154.3, 43.9)
- added U1: USBLC6-4SC6, Package_TO_SOT_SMD:SOT-23-6, F.Cu at (150.8, 67.1)
- added U10: ADS7822U, supercap:SOIC127P599X175-8N, F.Cu at (118.1, 81.1)
- added U11: TX4139, Package_SO:SOIC-8-1EP_3.9x4.9mm_P1.27mm_EP2.29x3mm_ThermalVias, F.Cu at (149.8, 43.2)
- added U12: TLV1117LV33DCYR, Package_TO_SOT_SMD:SOT-223-3_TabPin2, F.Cu at (161.0, 54.8)
- added U13: TXS0101DCKR, Package_TO_SOT_SMD:SOT-363_SC-70-6, F.Cu at (162.0, 109.9)
- added U14: EL357N(C)(TA)-G, Package_SO:SO-4_4.4x3.6mm_P2.54mm, F.Cu at (158.0, 93.3)
- added U2: W25Q128JVSIQ, Package_SO:SOIC-8_5.23x5.23mm_P1.27mm, F.Cu at (144.6, 74.0)
- added U3: ADC081S021CISD/NOPB, Package_TO_SOT_SMD:SOT-23-6, F.Cu at (95.3, 162.7)
- added U4: RP2040, RP2040_minimal:RP2040-QFN-56, F.Cu at (148.3, 86.2)
- added U5: ADC081S021CISD/NOPB, Package_TO_SOT_SMD:SOT-23-6, F.Cu at (85.8, 160.0)
- added U6: INA181A2, Package_TO_SOT_SMD:SOT-23-6, F.Cu at (158.1, 126.7)
- added U7: INA181A2, Package_TO_SOT_SMD:SOT-23-6, F.Cu at (79.1, 131.1)
- added U8: USBLC6-2P6, Package_TO_SOT_SMD:SOT-666, F.Cu at (158.1, 81.7)
- added U9: MT2492, Package_TO_SOT_SMD:SOT-23-6, F.Cu at (159.7, 36.1)
- added Y1: 12MHz, Crystal:Crystal_SMD_3225-4Pin_3.2x2.5mm, F.Cu at (147.7, 98.5)
- C10: renamed from C207; moved to B.Cu
- C12: renamed from C209; moved to B.Cu
- C17: renamed from C211; moved to B.Cu
- C19: renamed from C213; moved to B.Cu
- C21: renamed from C215; moved to B.Cu
- C23: renamed from C217; moved to B.Cu
- C25: renamed from C219; moved to B.Cu
- C27: renamed from C221; moved to B.Cu
- C5: renamed from C202; moved to B.Cu
- C7: renamed from C204; moved to B.Cu
- J3: renamed from J203; moved to F.Cu
- J5: renamed from J202; moved to F.Cu
- moved C26 74.9 mm to (72.0, 91.0)
- moved C8 73.8 mm to (129.0, 60.5), turned to 90 degrees
- moved C7 73.4 mm to (129.0, 79.5)
- moved C10 72.6 mm to (110.0, 34.0), turned to -90 degrees
- moved C22 72.1 mm to (91.0, 41.5)
- moved C23 71.8 mm to (72.0, 34.0)
- moved C27 65.3 mm to (72.0, 110.0), turned to -90 degrees
- moved C9 64.7 mm to (129.0, 41.5), turned to 90 degrees
- moved C13 62.9 mm to (110.0, 91.0), turned to -90 degrees
- moved C5 61.0 mm to (129.0, 117.5), turned to 90 degrees
- moved C6 57.8 mm to (129.0, 98.5)
- moved C19 54.8 mm to (91.0, 98.5), turned to 90 degrees
- moved C25 45.1 mm to (72.0, 72.0)
- moved J5 44.9 mm to (138.7, 137.7), turned to -90 degrees
- moved C18 41.4 mm to (91.0, 117.5)
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- renumbered C208 to C11, C210 to C13, C212 to C18, C214 to C20, C216 to C22, C218 to C24, C220 to C26, C203 to C6, C205 to C8, C206 to C9, Q204 to Q11, Q205 to Q13, Q206 to Q14, Q207 to Q15, Q201 to Q4, Q202 to Q5
Connections:
- net /VBUS_GATE renamed /VINPUT_GATE
- net VBUS renamed VINPUT
- J3 pad 2: GND -> Net-(J3-Pin_2)
- J5 pad 2: GND -> Net-(J4-Pin_2)
- Q11 pad 1: +5V -> VOUT_ENABLE
- Q4 pad 2: VCAP -> Net-(Q4-D)
- Q5 pad 2: VCAP -> Net-(Q5-D)
Routing:
- net +3V3: track 0.00 -> 465.6 mm, vias 0 -> 21
- net VCAP: track 0.00 -> 282.6 mm, vias 0 -> 21
- net VIN_ENABLE: track 0.00 -> 180.6 mm, vias 0 -> 4
- net /ADC_CLK: track 0.00 -> 179.5 mm, vias 0 -> 4
- net /ADC_DATA: track 0.00 -> 178.2 mm, vias 0 -> 2
- net VOUT_MEASURE: track 0.00 -> 156.6 mm, vias 0 -> 2
- net /ADC_CS1: track 0.00 -> 151.5 mm, vias 0 -> 2
- net /ADC_CS2: track 0.00 -> 138.2 mm
- net GND: track 0.00 -> 132.9 mm, vias 0 -> 144
- net CURRENT_MEASURE_OUT: track 0.00 -> 125.4 mm, vias 0 -> 2
- net +5V: track 0.00 -> 122.2 mm, vias 0 -> 9
- net /VINPUT_GATE: track 0.00 -> 104.2 mm
- net VINPUT: track 0.00 -> 97.7 mm, vias 0 -> 2
- net VOUT_ENABLE: track 0.00 -> 79.8 mm, vias 0 -> 2
- net Net-(J4-Pin_2): track 0.00 -> 77.6 mm, vias 0 -> 30
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- added copper zone on F.Cu, net +3V3
- added copper zone on F.Cu, net +5V
- added copper zone on F.Cu, net /1V1
- added copper zone on F.Cu, net GND
- added copper zone on In1.Cu, net GND
- added copper zone on In2.Cu, net GND
- added copper zone on F.Cu, net Net-(J3-Pin_2)
- added copper zone on F.Cu, net Net-(U9-SW)
- added copper zone on F.Cu, net VINPUT
- added copper zone on F.Cu, net VOUT
Other:
- board size 70 x 174 mm -> 109 x 155.5 mm
