File: supercap/supercap/supercap.kicad_sch (KiCad schematic)
At the start: 48 parts, among them J11 CAN2 PLUG, J201 Conn_01x02, J202 Conn_01x02, J203 Power Output, Q201 100V 34A PMOS, Q202 100V 34A PMOS, Q203 100V 34A PMOS, Q205 100V 34A PMOS, Q206 100V 34A PMOS, Q207 100V 34A PMOS, Q7 Q_NMOS_GSD

Commit message: Rev 2 Supercap PCB, updates to Motherboard in progress
Parts:
- removed C201, C222: 1uF, Capacitor_SMD:C_0805_2012Metric, symbol Device:C
- removed H201, H202: MountingHole_Pad, supercap:Sinhoo-SMTSO40x-C2916378, symbol Mechanical:MountingHole_Pad
- removed JP201, JP202, JP203, JP204, JP205, JP206, JP207: SolderJumper_2_Open, Jumper:SolderJumper-2_P1.3mm_Open_RoundedPad1.0x1.5mm, symbol Jumper:SolderJumper_2_Open
- removed Q203: 100V 34A PMOS, Package_TO_SOT_SMD:TO-252-2, symbol Device:Q_PMOS_GDS
- removed R201, R203: 10k, Resistor_SMD:R_0805_2012Metric, symbol Device:R
- removed R202, R204: 20k, Resistor_SMD:R_0805_2012Metric, symbol Device:R
- added C18, C20, C35, C406, C410, C415: 1u, Capacitor_SMD:C_0603_1608Metric, symbol Device:C
- added C22, C403, C404, C405, C407, C408 (x3), C409, C411, C412, C413, C414, C421: 100n, Capacitor_SMD:C_0603_1608Metric, symbol Device:C
- added C26: 47uF 63V solid, Capacitor_THT:CP_Radial_D8.0mm_P3.50mm, symbol Device:C_Polarized
- added C401, C402: 20p, Capacitor_SMD:C_0603_1608Metric, symbol Device:C
- added C417: 4.7uF 100V, Capacitor_SMD:C_1210_3225Metric, symbol Device:C
- added C418: 100nF 100V, Capacitor_SMD:C_0805_2012Metric, symbol Device:C
- added C419: 10u, Capacitor_SMD:C_0805_2012Metric, symbol Device:C
- added C420, C427: 22uF 25V, Capacitor_SMD:C_0805_2012Metric, symbol Device:C
- added C422: 47pf, Capacitor_SMD:C_0603_1608Metric, symbol Device:C
- added C423: 22nF, Capacitor_SMD:C_0603_1608Metric, symbol Device:C
- added C424: 220uF 25V, Capacitor_SMD:CP_Elec_6.3x7.7, symbol Device:C_Polarized
- added C425: 22pF, Capacitor_SMD:C_0603_1608Metric, symbol Device:C
- added C426: 47uF 10v, Capacitor_SMD:C_0805_2012Metric, symbol Device:C
- added D10, D11, D12, D13, D14, D15, D16, D17, D18, D19, D2, D20, D21, D3, D4, D5, D6, D7, D8, D9: 2.4v zener, supercap:DIO_PESD5V0S1UL_315, symbol Device:D_Zener
- added D23, D25: D, Diode_SMD:D_SMA, symbol Device:D
- added D31 (x3): 1N4148WS, Diode_SMD:D_SOD-323, symbol Device:D
- added D33, D34: Zener 10v, Diode_SMD:D_SOD-323, symbol Device:D_Zener
- added D33, D34, D35: WS2812B, RP2040_minimal:LED_WS2812_3528_3.5x2.8mm_P1.5mm, symbol MotorBuck:WS2812B
- added D401: B5819W SL, Diode_SMD:D_SOD-123, symbol Diode:MBR340
- added D402 (x2): SMAJ51A, Diode_SMD:D_SMA, symbol Diode:SMF54A
- added D403: SS310, Diode_SMD:D_SMA, symbol Diode:MBR340
- added H8 (x2): MountingHole, supercap:MountingHole_3.9mm_Plastite_#6, symbol Mechanical:MountingHole
- added J401: CPU2 USB, Connector_USB:USB_C_Receptacle_XKB_U262-16XN-4BVC11, symbol Connector:USB_C_Receptacle_USB2.0
- added J402: Conn_01x06, parts:Ckmtw-W-2510S06P_1x06_P2.54mm_Vertical, symbol Connector_Generic:Conn_01x06
- added JP1, JP10, JP2, JP3, JP4, JP5, JP6, JP7, JP8, JP9: SolderJumper_2_Open, Jumper:SolderJumper-2_P1.3mm_Open_RoundedPad1.0x1.5mm, symbol Jumper:SolderJumper_2_Open
- added L401: 47uH, Inductor_SMD:L_Chilisin_BMRB00060612, symbol Device:L
- added L402: 10uH, Inductor_SMD:L_Sunlord_SWPA5040S, symbol Device:L
- added Q12, Q2, Q3, Q6, Q7, Q8, Q9: 100V 34A PMOS, Package_TO_SOT_SMD:TO-252-2, symbol Device:Q_PMOS_GDS
- added Q7 (x2): Q_NMOS_GSD, Package_TO_SOT_SMD:SOT-23, symbol Device:Q_NMOS_GSD
- added R1, R24: 10k, Resistor_SMD:R_1206_3216Metric, symbol Device:R
- added R101 (x2), R116: 3mΩ, Resistor_SMD:R_2512_6332Metric, symbol MotorController:TAYLOR_RESISTOR
- added R16, R17, R18, R19, R20, R21, R22, R23: 100R 2W, Resistor_SMD:R_2512_6332Metric, symbol Device:R
- added R2, R3: 1k 2 watt, Resistor_SMD:R_2512_6332Metric, symbol Device:R
- added R2 (x3), R64 (x3): 50k 0.1%, Resistor_SMD:R_0603_1608Metric, symbol MotorController:TAYLOR_RESISTOR
- added R21, R45: 10k, Resistor_SMD:R_0603_1608Metric, symbol MotorController:TAYLOR_RESISTOR
- added R40, R41: 2k 2 watt, Resistor_SMD:R_2512_6332Metric, symbol Device:R
- added R401, R405: 1.1k, Resistor_SMD:R_0603_1608Metric, symbol Device:R
- added R402: DNS, Resistor_SMD:R_0402_1005Metric, symbol Device:R
- added R403, R404, R76: 5.1k, Resistor_SMD:R_0603_1608Metric, symbol Device:R
- added R406, R407: 27, Resistor_SMD:R_0603_1608Metric, symbol Device:R
- added R408: 50mΩ, Resistor_SMD:R_0603_1608Metric, symbol Device:R
- added R409: 10Ω, Resistor_SMD:R_0603_1608Metric, symbol Device:R
- added R410: 300k, Resistor_SMD:R_0603_1608Metric, symbol Device:R
- added R411: 21.5k, Resistor_SMD:R_0603_1608Metric, symbol Device:R
- added R412: 110k 0.1%, Resistor_SMD:R_0603_1608Metric, symbol Device:R
- added R413: 15k 0.1%, Resistor_SMD:R_0603_1608Metric, symbol Device:R
- added R65 (x3): 5.1k 0.1%, Resistor_SMD:R_0603_1608Metric, symbol MotorController:TAYLOR_RESISTOR
- added R75: 120R, Resistor_SMD:R_0603_1608Metric, symbol MotorController:TAYLOR_RESISTOR
- added SW401 (x4): SW_MEC_5G, supercap:SW_TS_1101_C_W, symbol Switch:SW_Push
- added TH1, TH2: Thermistor 10k, Resistor_SMD:R_0603_1608Metric, symbol Device:Thermistor_NTC
- added TP401: TestPoint, TestPoint:TestPoint_Loop_D2.60mm_Drill1.6mm_Beaded, symbol Connector:TestPoint
- added TP402, TP403, TP404: TestPoint, TestPoint:TestPoint_Pad_D2.0mm, symbol Connector:TestPoint
- added U10: TXS0101DCKR, Package_TO_SOT_SMD:SOT-363_SC-70-6, symbol MotorBuck:level_shifter
- added U21: EL357N(C)(TA)-G, Package_SO:SO-4_4.4x3.6mm_P2.54mm, symbol Isolator:LTV-357T
- added U22: ADS7822U, supercap:SOIC127P599X175-8N, symbol ADS7822U:ADS7822U
- added U26, U9: ADC081S021CISD/NOPB, Package_TO_SOT_SMD:SOT-23-6, symbol 2022-06-16_01-48-54:ADC081S021CISD/NOPB
- added U401: USBLC6-4SC6, Package_TO_SOT_SMD:SOT-23-6, symbol Power_Protection:USBLC6-4SC6
- added U402: W25Q128JVSIQ, Package_SO:SOIC-8_5.23x5.23mm_P1.27mm, symbol Memory_Flash:W25Q128JVS
- added U403: RP2040, RP2040_minimal:RP2040-QFN-56, symbol MCU_RaspberryPi_RP2040:RP2040
- added U404: USBLC6-2P6, Package_TO_SOT_SMD:SOT-666, symbol Power_Protection:USBLC6-2P6
- added U405: TLV1117LV33DCYR, Package_TO_SOT_SMD:SOT-223-3_TabPin2, symbol Regulator_Linear:NCP1117-3.3_SOT223
- added U406: TX4139, Package_SO:SOIC-8-1EP_3.9x4.9mm_P1.27mm_EP2.29x3mm_ThermalVias, symbol MotorBuck:TX4139
- added U407: MT2492, Package_TO_SOT_SMD:SOT-23-6, symbol Regulator_Switching:AP3211K
- added U6, U7: INA181A2, Package_TO_SOT_SMD:SOT-23-6, symbol Amplifier_Current:INA181
- added Y401: 12MHz, Crystal:Crystal_SMD_3225-4Pin_3.2x2.5mm, symbol Device:Crystal_GND24
- Q7: LCSC C400505 -> C2891566
- renumbered C207 to C10, C208 to C11, C209 to C12, C210 to C13, C211 to C17, C212 to C18, C213 to C19, C214 to C20, C215 to C21, C216 to C22, C217 to C23, C218 to C24, C219 to C25, C220 to C26, C221 to C27, C202 to C5, C203 to C6, C204 to C7, C205 to C8, C206 to C9, J203 to J3, J201 to J4, J202 to J5, Q205 to Q13, Q206 to Q14, Q207 to Q15, Q201 to Q4, Q202 to Q5
Connections:
- net +5V: now also C415.1, C425.1, C426.2, C427.2, D33.3 (VDD), D34.3 (VDD), D35.3 (VDD), D401.1 (K), L402.2, R412.2, U10.6 (VCCB), U405.3 (VI); no longer J11.1 (Pin_1), Q7.1 (G)
- net GND: now also C18.1, C20.1, C22.2, C26.2, C35.1, C401.2, C402.2, C403.2, C404.2, C405.2, C406.2, C407.2, C408.2, C408.2, C408.2, C409.2, C410.2, C411.2, C412.2, C413.2, C414.2, C415.2, C417.2, C418.2, C419.2, C420.2, C424.2, C426.1, C427.1, D21.2 (A), D33.1 (GND), D34.1 (GND), D35.1 (GND), D402.2 (A2), D402.2 (A2), D403.2 (A), J401.A1 (GND), J401.A12 (GND), J401.B1 (GND), J401.B12 (GND), J401.S1 (SHIELD), J402.6 (Pin_6), Q7.2 (S), Q7.2 (S), R101.1, R101.1, R116.1, R21.2, R403.1, R404.2, R411.1, R413.2, R45.2, R65.2, R65.2, R65.2, SW401.1, SW401.2, SW401.2, SW401.2, TP401.1, U10.2 (GND), U21.3, U22.3 (IN-), U22.4 (GND), U26.2 (GND), U401.2 (GND), U402.4 (GND), U403.19 (TESTEN), U403.57 (GND), U404.2 (GND), U405.1 (GND), U406.4 (GND), U407.2 (GND), U6.2 (GND), U6.4 (-), U6.5 (REF), U7.2 (GND), U7.4 (-), U7.5 (REF), U9.2 (GND), Y401.2, Y401.4; no longer J11.4 (Pin_4), J3.2 (Pin_2), J4.2 (Pin_2), J5.2 (Pin_2)
- net VBUS: now also D25.2 (A), D401.2 (A), J401.A4 (VBUS), J401.A9 (VBUS), J401.B4 (VBUS), J401.B9 (VBUS), U404.5 (VBUS); no longer J4.1 (Pin_1), J5.1 (Pin_1), Q4.3 (S), Q5.3 (S)
- net VCAP: now also D2.1 (K), D23.2 (A), D34.1 (K), JP1.2 (B), JP10.1 (A), JP2.2 (B), JP3.2 (B), JP4.2 (B), JP5.2 (B), JP6.1 (A), JP7.1 (A), JP8.1 (A), JP9.1 (A), Q12.3 (S), Q6.3 (S), Q7.3 (S), Q8.3 (S), Q9.3 (S), R16.1, R17.1, R2.1, R2.2, R24.1, R3.2; no longer Q4.2 (D), Q5.2 (D)
- net VCAP_GATE: now also D34.2 (A), Q12.1 (G), R24.2, R41.2
- net VOUT: now also D402.1 (A1), JP10.2 (B), JP6.2 (B), JP7.2 (B), JP8.2 (B), JP9.2 (B), Q12.2 (D), R2.1
- net at C11.2, C12.1: now also D8.2 (A), D9.1 (K)
- net at C12.2, C13.1: now also D10.1 (K), D9.2 (A)
- net at C24.2, C25.1: now also D18.2 (A), D19.1 (K)
- net at C25.2, C26.1: now also D19.2 (A), D20.1 (K)
- net at C26.2, C27.1: now also D20.2 (A), D21.1 (K)
- net at C13.2, C17.1: now also D10.2 (A), D11.1 (K)
- net at Q7.3 (D): now also R41.1
- net at C10.1, C9.2: now also D6.2 (A), D7.1 (K)
- net at C10.2, C11.1: now also D7.2 (A), D8.1 (K)
- net at C17.2, C18.1: now also D11.2 (A), D12.1 (K)
- net at C18.2, C19.1: now also D12.2 (A), D13.1 (K)
- net at C19.2, C20.1: now also D13.2 (A), D14.1 (K)
- net at C23.2, C24.1: now also D17.2 (A), D18.1 (K)
- net at C5.2, C6.1: now also D2.2 (A), D3.1 (K)
- net at C21.2, C22.1: now also D15.2 (A), D16.1 (K)
- net at C22.2, C23.1: now also D16.2 (A), D17.1 (K)
- net at C20.2, C21.1: now also D14.2 (A), D15.1 (K)
- net at C6.2, C7.1: now also D3.2 (A), D4.1 (K)
- net at C7.2, C8.1: now also D4.2 (A), D5.1 (K)
- net at C8.2, C9.1: now also D5.2 (A), D6.1 (K)
- net VBUS_GATE renamed VINPUT_GATE
- net VINPUT_GATE: now also D33.2 (A), Q2.1 (G), Q3.1 (G), Q6.1 (G), Q7.1 (G), Q8.1 (G), Q9.1 (G), R1.2, R40.2
- new net: R16.2, R18.1
- new net: R18.2, R20.1
- new net: R21.1, TH2.2, U26.3 (VIN)
- new net: Q4.2 (D), Q8.2 (D)
- new net: C26.1, C417.1, C418.1, D23.1 (K), D25.1 (K), R408.2, U406.3 (VIN)
- new net: Q3.2 (D), Q7.2 (D)
- new net: J401.A5 (CC1), R403.2
- new net: J401.B5 (CC2), R404.1
- new net: J3.2 (Pin_2), R101.2, R116.2, U7.3 (+)
- new net: R17.2, R19.1
- new net: R19.2, R21.1
- new net: J4.2 (Pin_2), J5.2 (Pin_2), R101.2, U6.3 (+)
- new net: C423.1, U407.1 (BS)
- new net: C425.2, R412.1, R413.1, U407.3 (FB)
- new net: C423.2, L402.1, U407.6 (SW)
- new net: R45.1, TH1.2, U9.3 (VIN)
- new net: SW401.1, U403.14 (GPIO11)
- new net: R20.2, R22.1
- new net: Q7.3 (D), R22.2, R23.2
- new net: C401.1, U403.20 (XIN), Y401.3
- new net: R408.1, U406.2 (ILIM), U406.9 (ILIM)
- new net: Q7.3 (D), R40.1
- new net: R2.2, R64.1 (x3)
- new net: Q2.2 (D), Q6.2 (D)
- new net: D31.2 (A), R64.2, R65.1, U22.2 (IN+)
- new net: R405.1, U403.21 (XOUT)
- new net: C402.1, R405.2, Y401.1
- new net: SW401.1, U403.12 (GPIO9)
- new net: SW401.1, U403.13 (GPIO10)
- new net: D33.2 (DIN), U10.4 (B)
- new net: C421.2, R409.2
- new net: R21.2, R23.1
- new net: R406.1, U404.1 (I/O1)
- new net: R407.1, U404.3 (I/O2)
- new net: Q5.2 (D), Q9.2 (D)
- new net: D33.4 (DOUT), D34.2 (DIN)
- new net: D34.4 (DOUT), D35.2 (DIN)
- new net: R75.2, U21.1
- new net +12V: C420.1, C422.1, C424.1, L401.2, R410.2, TP404.1, U407.4 (EN), U407.5 (IN)
- new net +3V3: C18.2, C20.2, C22.1, C35.2, C403.1, C407.1, C408.1, C408.1, C408.1, C409.1, C410.1, C411.1, C412.1, C413.1, C414.1, C419.1, D31.1 (K), D31.1 (K), D31.1 (K), J402.3 (Pin_3), R402.1, R76.1, TH1.1, TH2.1, U10.1 (VCCA), U10.5 (OE), U22.1 (VREF), U22.8 (+VCC), U26.1 (VA), U401.5 (VBUS), U402.8 (VCC), U403.1 (IOVDD), U403.10 (IOVDD), U403.22 (IOVDD), U403.26 (RUN), U403.33 (IOVDD), U403.42 (IOVDD), U403.43 (ADC_AVDD), U403.44 (VREG_IN), U403.48 (USB_VDD), U403.49 (IOVDD), U405.2 (VO), U6.6 (V+), U7.6 (V+), U9.1 (VA)
- new net +5V_ISO: J11.1 (Pin_1), R75.1
- new net 1V1: C404.1, C405.1, C406.1, U403.23 (DVDD), U403.45 (VREG_VOUT), U403.50 (DVDD)
- new net 5V_ISO_PRESENT: R76.2, U21.4, U403.28 (GPIO17)
- new net ADC_CLK: U22.7 (DCLK), U26.4 (SCLK), U403.4 (GPIO2), U9.4 (SCLK)
- new net ADC_CS1: U403.3 (GPIO1), U9.6 (~{CS})
- new net ADC_CS2: U26.6 (~{CS}), U403.5 (GPIO3)
- new net ADC_CS3: U22.5 (~{CS/SHDN}), U403.6 (GPIO4)
- new net ADC_DATA: U22.6 (DOUT), U26.5 (SDATA), U403.2 (GPIO0), U9.5 (SDATA)
- new net BLEED_FET: Q7.1 (G), U403.8 (GPIO6)
- new net BS: R409.1, U406.8 (BS)
- new net CURRENT_MEASURE_IN: U403.38 (GPIO26_ADC0), U6.1
- new net CURRENT_MEASURE_OUT: U403.39 (GPIO27_ADC1), U7.1
- new net FB: C422.2, R410.1, R411.2, U406.5 (FB)
- new net GND_ISO: J11.4 (Pin_4), U21.2
- new net LED: U10.3 (A), U403.7 (GPIO5)
- new net QSPI_SCLK_2: U402.6 (CLK), U403.52 (QSPI_SCLK)
- new net QSPI_SD0_2: U402.5 (DI(IO0)), U403.53 (QSPI_SD0)
- new net QSPI_SD1_2: U402.2 (DO(IO1)), U403.55 (QSPI_SD1)
- new net QSPI_SD2_2: U402.3 (IO2), U403.54 (QSPI_SD2)
- new net QSPI_SD3_2: U402.7 (IO3), U403.51 (QSPI_SD3)
- new net QSPI_SS_2: R401.1, R402.2, U402.1 (~{CS}), U403.56 (QSPI_SS)
- new net RXI_2: J402.4 (Pin_4), U401.4 (I/O3), U403.37 (GPIO25)
- new net SW: C421.1, D403.1 (K), L401.1, U406.1 (SW)
- new net SWCLK_2: J402.1 (Pin_1), U401.3 (I/O2), U403.24 (SWCLK)
- new net SWD_2: J402.2 (Pin_2), U401.1 (I/O1), U403.25 (SWD)
- new net TXO_2: J402.5 (Pin_5), U401.6 (I/O4), U403.36 (GPIO24)
- new net USB_DN_2: R407.2, U403.46 (USB_DM)
- new net USB_DP_2: R406.2, U403.47 (USB_DP)
- new net USB_D_2+: J401.A6 (D+), J401.B6 (D+), TP403.1, U404.6 (I/O1)
- new net USB_D_2-: J401.A7 (D-), J401.B7 (D-), TP402.1, U404.4 (I/O2)
- new net VINPUT: D33.1 (K), D402.1 (A1), J4.1 (Pin_1), J5.1 (Pin_1), JP1.1 (A), JP2.1 (A), JP3.1 (A), JP4.1 (A), JP5.1 (A), Q2.3 (S), Q3.3 (S), Q4.3 (S), Q5.3 (S), R1.1, R2.1, R2.1, R3.1
- new net VINPUT_MEASURE: D31.2 (A), R64.2, R65.1, U403.40 (GPIO28_ADC2)
- new net VIN_ENABLE: Q7.1 (G), U403.11 (GPIO8)
- new net VOUT_ENABLE: Q7.1 (G), U403.9 (GPIO7)
- new net VOUT_MEASURE: D31.2 (A), R64.2, R65.1, U403.41 (GPIO29_ADC3)
- new net ~{USB_BOOT_2}: R401.2, SW401.2
Other:
- note added: "11.7-12.3V 800mA"
- note added: "4.9-5.1V"
- note added: "CPU"
- note added: "Capacitor Voltage Sense"
- note added: "Crystal"
- note added: "Debug"
- note added: "Flash"
- note added: "Internal pullup on EN"
- note added: "Make sure C54 is close to pin 44 of RP2040"
- note added: "Make sure C8 is close to pin 45 of RP2040"
- note added: "Onboard Thermistors"
- note added: "Power"
- note added: "R_{ILIM} 50mohm = 0.8A Iout max I_{In} = 400mA max => 8mW max Pd"
- note added: "TVS protection"
- moved on the sheet: C10, C11, C12, C13, C17, C18, C19, C20, C21, C22, C23, C24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
