File: cm4_robot_board/cm4-robot.kicad_sch (KiCad schematic)
At the start: 157 parts, among them J1 1747981-1, J10 Conn_01x04, J11 Conn_01x03, J12 Conn_01x04, J13 RJ45, J14 RJ45, J15 RJ45, J16 RJ45, J17 Conn_01x04, J18 Conn_01x04, J19 Conn_01x04, J2 HR913550A, J20 Conn_01x04, J21 Conn_01x03, J22 Conn_01x04, J23 Conn_01x01, J24 Conn_01x01, J3 USB_C_Receptacle_USB2.0, J4 Conn_01x04, J5 Conn_01x04, J6 Conn_01x04, J7 USB_A, J8 HIGHCURRENTPAD2, J9 HIGHCURRENTPAD2, Q1 Q_PMOS_GSD, Q2 Q_NMOS_GSD, Q3 Q_NMOS_GSD, Q4 Q_NMOS_GSD, Q5 Q_NMOS_GSD, SW1 B3U-1000P, SW2 SW_SPDT, SW3 SW_SPDT, U1 SN74LVC1G07QDCKTQ1, U10 isolator, U11 isolator, U12 TPS61040DBVR, U13 SC16IS752, U14 SC16IS752, U15 SN74LVC1G07QDCKTQ1, U16 CC56-12SEKWA, U17 ET6226M, U18 SN74LVC1G07QDCKTQ1, U19 SN74LVC1G07QDCKTQ1, U2 SN74LVC1G07QDCKTQ1, U3 LM2576HVS-5, U4 TPD4E1U06DCKR, U5 ISL54222AIUZ, U6 LTC4412xS6, U7 SN74HC08N, U8 MCP2515-xSO, U9 MCP2515-xSO, Y1 Crystal_GND24, Y2 Crystal_GND24, Y3 Crystal_GND24, Y4 Crystal_GND24

Commit message: Update latest files for CM4 robot board. Ordered this version.
Parts:
- removed C17: 1000uF, Capacitor_SMD:CP_Elec_10x10, symbol Device:C_Polarized
- removed D12, D13, D14, D15: D_TVS, Diode_SMD:D_SOD-323, symbol Device:D_TVS
- removed D16: LED_GREEN, LED_SMD:LED_0805_2012Metric, symbol Device:LED
- removed J15, J16: RJ45, Connector_RJ:RJ45_OST_PJ012-8P8CX_Vertical, symbol Connector:RJ45
- removed JP5, JP6, JP7, JP8: SolderJumper_2_Open, Jumper:SolderJumper-2_P1.3mm_Open_RoundedPad1.0x1.5mm, symbol Jumper:SolderJumper_2_Open
- removed R15: 10k, Resistor_SMD:R_0603_1608Metric, symbol MotorController:TAYLOR_RESISTOR
- removed R23: 220R, Resistor_SMD:R_0603_1608Metric, symbol Device:R
- removed R30, R31, R32, R33: 1k, Resistor_SMD:R_0603_1608Metric, symbol Device:R
- removed U7: SN74HC08N, Package_SO:SOIC-14_3.9x8.7mm_P1.27mm, symbol dk_Logic-Gates-and-Inverters:SN74HC08N
- added D12: LED_GREEN, LED_SMD:LED_0805_2012Metric, symbol Device:LED
- added JP1, JP2: SolderJumper_2_Open, Jumper:SolderJumper-2_P1.3mm_Open_RoundedPad1.0x1.5mm, symbol Jumper:SolderJumper_2_Open
- added R15: 56R, Resistor_SMD:R_0603_1608Metric, symbol Device:R
- added R23, R30: 10k, Resistor_SMD:R_0603_1608Metric, symbol MotorController:TAYLOR_RESISTOR
- added TP2: TestPoint, TestPoint:TestPoint_Keystone_5019_Minature, symbol Connector:TestPoint
- added U7: TXS0101DCKR, Package_TO_SOT_SMD:SOT-363_SC-70-6, symbol 2022-12-10_08-30-32:TXS0101DCKR
- C10, C4, C7, C8: value 10p -> 18p; LCSC C106245 -> C1647
- C11: value 10uF -> 0.1uF; footprint Capacitor_SMD:C_0805_2012Metric -> Capacitor_SMD:C_0603_1608Metric; Digikey 311-1355-1-ND -> (none); LCSC C15850 -> C14663; MPN CC0805ZKY5V6BB106 -> (none)
- C18: value 10uF -> 4.7uF; LCSC C92487 -> C69335
- C19: value 4.7pF -> 2.7pF; LCSC C1669 -> C95180
- C20: value 4.7uF -> 1uF; LCSC C69335 -> C59302
- C21, C22, C23, C24: value 12pF -> 22p; LCSC C107034 -> C1653
- D18, D19, D20, D21, D5, D6, D7: LCSC C2920042 -> C2761795
- D3: footprint Diode_SMD:D_SMB -> Diode_SMD:D_SMA; LCSC C13762 -> C15874
- J13, J14: footprint Connector_RJ:RJ45_OST_PJ012-8P8CX_Vertical -> parts:RJ45_R-RJ45R08P-B000; LCSC C2902702 -> C386756
- L1: footprint parts:MWSA1206S-680MT -> parts:L_15mmx15mm; LCSC C408533 -> C970545
- R13: value 220R -> 27R; Digikey A129741CT-ND -> (none); LCSC C22962 -> C25190
Connections:
- net E2B is gone; now on net +3V3: R28.1
- net E3B is gone; now on net ESTOP_SINK: J14.5
- net E4B is gone; now on net +3V3: R14.1
- net +3V3: now also R29.1, R23.1, R30.1, U7.1 (VCCA), U7.5 (OE); no longer C11.1, D18.1 (VDD), D19.1 (VDD), D20.1 (VDD), D21.1 (VDD), D5.1 (VDD), D6.1 (VDD), D7.1 (VDD), J21.1 (Pin_1)
- net +5V: now also C11.1, D18.1 (VDD), D19.1 (VDD), D20.1 (VDD), D21.1 (VDD), D5.1 (VDD), D6.1 (VDD), D7.1 (VDD), J21.1 (Pin_1), U7.6 (VCCB)
- net CANH0: now also JP2.1 (A); no longer R34.1
- net CANH1: now also JP1.1 (A); no longer R35.1
- net CANL0: now also R34.1; no longer R34.2
- net CANL1: now also R35.1; no longer R35.2
- net ESTOP: now also U15.2 (A)
- net ESTOP_OUT: now also D8.2 (A)
- net GND: now also J24.1 (Pin_1), R13.1, R15.1, TP2.1, U7.2 (GND); no longer R13.2, R14.2, R28.2, R29.2, U15.1 (/OE)
- net SCL0_GPIO45: now also R28.2
- net SCL6: now also R29.2
- net SDA0_GPIO44: now also R23.2
- net SDA6: now also R30.2
- net TRD0_N: now also U4.6 (CH4); no longer U4.3 (CH2)
- net TRD1_N: now also U4.3 (CH2); no longer U4.4 (CH3)
- net TRD1_P: now also U4.4 (CH3); no longer U4.6 (CH4)
- net WS2812: now also U7.3 (A); no longer D5.4 (DIN)
- net at D17.1 (K): now also R15.2
- net at U18.4 (Y): now also D12.2 (A)
- net E1B renamed ESTOP_SINK
- net ESTOP_SINK: now also R14.2, U15.1 (/OE); no longer R29.1
- new net: JP1.2 (B), R35.2
- new net: D12.1 (K), R13.2
- new net: D5.4 (DIN), U7.4 (B)
- new net: JP2.2 (B), R34.2
- no-connect marks 33 -> 35
Other:
- note added: "Dummy parts for Hirose connector placement. To be placed on top of CM4 connectors."
- note added: "SPI naming note: I wanted to move away from master/slave naming but in doing so I used inconsistent and unclear conventions. -TLA TODO: Use "primary/secondary" and make everything PISO/POSI"
- note added: "TODO: FIX SPI NAMING POSI PISO (primary/secondary)"
- note removed: "Estop Bypass Jumpers"
- note removed: "MOTOR1"
- note removed: "MOTOR2"
- note removed: "MOTOR3"
- note removed: "MOTOR4"
- moved on the sheet: D18, D19, D20, D21, D5, D6, D7, D8, J13, J14, J21, R27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

Commit message: Rev 2 Supercap PCB, updates to Motherboard in progress
Parts:
- removed C1: 0.1uF, Capacitor_SMD:C_0603_1608Metric, symbol Device:C
- removed J13, J14: RJ45, parts:RJ45_R-RJ45R08P-B000, symbol Connector:RJ45
- removed J2: HR913550A, HANRUN_HR911105A, symbol HR911105A:HR911105A
- removed R14: 10k, Resistor_SMD:R_0603_1608Metric, symbol MotorController:TAYLOR_RESISTOR
- added C20, C23: 10u, Capacitor_SMD:C_0805_2012Metric, symbol Device:C
- added C26: 47uF 63V solid, Capacitor_THT:CP_Radial_D8.0mm_P3.50mm, symbol Device:C_Polarized
- added C33, C38: 47uF 16V, Capacitor_SMD:C_1210_3225Metric, symbol Device:C
- added C34: 22pF, Capacitor_SMD:C_0603_1608Metric, symbol Device:C
- added C35: 22uF 10v, Capacitor_SMD:C_0805_2012Metric, symbol Device:C
- added C36, C37: 22uF 6.3v, Capacitor_SMD:C_0603_1608Metric, symbol Device:C
- added C39: 0.1uF, Capacitor_SMD:C_0805_2012Metric, symbol Device:C
- added C42, C44, C45, C46: 22nF 100v, Capacitor_SMD:C_0603_1608Metric, symbol Device:C
- added C43: 1nF 2kV, Capacitor_SMD:C_1206_3216Metric, symbol Device:C
- added C47: 0.1uF, Capacitor_SMD:C_0603_1608Metric, symbol Device:C
- added D13, D22: ABS2, Diode_SMD:Diode_Bridge_Diotec_ABS, symbol Diode_Bridge:ABS2
- added D14: LED_GREEN, LED_SMD:LED_0805_2012Metric, symbol Device:LED
- added D15: SMAJ60A, Diode_SMD:D_SMA, symbol Diode:SMAJ60A
- added D16: D, Diode_SMD:D_SMA, symbol Device:D
- added D23: LED_YELLOW, LED_SMD:LED_0805_2012Metric, symbol Device:LED
- added D24: 28V / 500mW, Diode_SMD:D_SOD-123, symbol Device:D_Zener
- added D25: 15V / 200mW, Diode_SMD:D_SOD-323, symbol Device:D_Zener
- added J14: Conn_01x03, Connector_Molex:Molex_KK-254_AE-6410-03A_1x03_P2.54mm_Vertical, symbol Connector_Generic:Conn_01x03
- added J15: Conn_02x04_Odd_Even, Connector_PinHeader_2.54mm:PinHeader_2x04_P2.54mm_Vertical, symbol Connector_Generic:Conn_02x04_Odd_Even
- added J2 (x2): CAN Interface, parts:M12A-08PFFR, symbol motor_parts:M12_X8_CONNECTOR
- added J25: RJ45, parts:RJ45_R-RJ45R08P-B000, symbol Connector:RJ45
- added JP5: SolderJumper_2_Open, Jumper:SolderJumper-2_P1.3mm_Open_RoundedPad1.0x1.5mm, symbol Jumper:SolderJumper_2_Open
- added L3: 10uH, Inductor_SMD:L_Sunlord_SWPA5040S, symbol Device:L
- added Q6: AO3401A, Package_TO_SOT_SMD:SOT-23, symbol Transistor_FET:AO3401A
- added Q7: AO3400A, Package_TO_SOT_SMD:SOT-23, symbol Transistor_FET:AO3400A
- added Q8: Si2328DS, Package_TO_SOT_SMD:SOT-23-3, symbol taylor_kicad:Q_NMOS_GSD
- added R14, R32: R, symbol Device:R
- added R33: 2.2k 1%, Resistor_SMD:R_0603_1608Metric, symbol Device:R
- added R36: 24.1k/1%, Resistor_SMD:R_0805_2012Metric, symbol Device:R
- added R37: 249k, Resistor_SMD:R_0805_2012Metric, symbol Device:R
- added R40: 51k, Resistor_SMD:R_0805_2012Metric, symbol Device:R
- added R41, R42, R43, R44: 75R 100v, Resistor_SMD:R_0603_1608Metric, symbol Device:R
- added R77: 82R, Resistor_SMD:R_0603_1608Metric, symbol MotorController:TAYLOR_RESISTOR
- added SW4: SW_SPDT, parts:CS12ANW03, symbol Switch:SW_SPDT
- added TR1: G2401CG, Transformer_SMD:Transformer_Ethernet_YDS_30F-51NL_SO-24_7.1x15.1mm, symbol Transformer:30F-51NL
- added U13: NCP1117-3.3_SOT223, Package_TO_SOT_SMD:SOT-223-3_TabPin2, symbol Regulator_Linear:NCP1117-3.3_SOT223
- added U22: MT2492, Package_TO_SOT_SMD:SOT-23-6, symbol Regulator_Switching:AP3211K
- added U23: TPD4E1U06DCKR, Package_TO_SOT_SMD:SOT-363_SC-70-6, symbol 2021-10-21_05-38-11:AOZ8904CIL
- C19: value 2.7pF -> 22pF; LCSC C95180 -> C1653
- D18, D19, D20, D21, D5, D6, D7: footprint LED_SMD:LED_WS2812B_PLCC4_5.0x5.0mm_P3.2mm -> parts:LED_WS2812B_PLCC4_5.0x5.0mm_P3.2mm
- D3: footprint Diode_SMD:D_SMA -> Diode_SMD:D_SMC; LCSC C15874 -> C123944
- R4: value 220R -> 2.2k 1%; Digikey A129741CT-ND -> RMCF0805FT2K10CT-ND; LCSC C22962 -> C4190; MPN (none) -> RMCF0805FT2K10
- TP2: footprint TestPoint:TestPoint_Keystone_5019_Minature -> TestPoint:TestPoint_Loop_D2.60mm_Drill1.6mm_Beaded; LCSC C238130 -> C5199814
- U7: LCSC (none) -> C132031
- Y1, Y2: value Crystal_GND24 -> 16MHz
- Y3, Y4: value Crystal_GND24 -> 14.7456MHz
Connections:
- net +3V3: now also R4.2, C23.1, D14.2 (A), D23.2 (A), JP5.1 (A), U13.2 (VO); no longer D1.2 (A), Module1.84 (+3.3v_(Output)), Module1.86 (+3.3v_(Output))
- net +5V: now also C20.1, C33.1, C35.1, C38.1, Q6.2 (S), R33.1, U22.5 (IN); no longer D2.2 (A)
- net ESTOP_OUT: now also J2.6 (Pin_6), J2.6 (Pin_6)
- net ESTOP_SINK: now also R4.1, J2.1 (Pin_1), J2.1 (Pin_1)
- net GND: now also C20.2, C23.2, C26.2, C33.2, C35.2, C38.2, C43.2, C47.1, J14.3 (Pin_3), J15.4 (Pin_4), J15.8 (Pin_8), J2.4 (Pin_4), J2.4 (Pin_4), J2.9, J2.9, Q7.2 (S), Q8.3 (D), R77.2, SW4.1 (A), U13.1 (GND), U22.2 (GND), U23.2 (VN); no longer R13.1, R15.1, R4.2, U3.5 (~{ON}/OFF)
- net TRD0_N: now also TR1.3 (TD1-)
- net TRD0_P: now also TR1.2 (TD1+)
- net TRD1_N: now also TR1.6 (TD2-)
- net TRD1_P: now also TR1.5 (TD2+)
- net VMOT: now also D16.1 (K), J15.2 (Pin_2), J15.6 (Pin_6)
- net at D2.1 (K): now also R77.1; no longer R4.1
- net at R3.1: now also D23.1 (K)
- net at R2.1: now also D14.1 (K)
- net at R13.2: now also D12.2 (A); no longer D12.1 (K)
- net at U18.4 (Y): now also D12.1 (K); no longer D12.2 (A)
- net at U19.4 (Y): now also D17.1 (K); no longer D17.2 (A)
- net at R15.2: now also D17.2 (A); no longer D17.1 (K)
- net TRD2_P: now reaches Module1.11 (Ethernet_Pair2_P)
- net TRD2_P: now also TR1.8 (TD3+), U23.1 (CH1)
- net TRD3_P: now reaches Module1.3 (Ethernet_Pair3_P)
- net TRD3_P: now also TR1.11 (TD4+), U23.4 (CH3)
- net TRD3_N: now reaches Module1.5 (Ethernet_Pair3_N)
- net TRD3_N: now also TR1.12 (TD4-), U23.3 (CH2)
- net TRD2_N: now reaches Module1.9 (Ethernet_Pair2_N)
- net TRD2_N: now also TR1.9 (TD3-), U23.6 (CH4)
- net CANH0 renamed CAN0_P
- net CAN0_P: now also J2.5 (Pin_5), J2.5 (Pin_5)
- net CANH1 renamed CAN1_P
- net CAN1_P: now also J2.2 (Pin_2), J2.2 (Pin_2)
- net CANL0 renamed CAN0_N
- net CAN0_N: now also J2.8 (Pin_8), J2.8 (Pin_8)
- net CANL1 renamed CAN1_N
- net CAN1_N: now also J2.3 (Pin_3), J2.3 (Pin_3)
- new net: C45.2, R43.1
- new net: C46.2, R44.1
- new net: C43.1, R41.2, R42.2, R43.2, R44.2
- new net: Q6.1 (G), Q7.3 (D), R33.2
- new net: C42.2, R41.1
- new net: C47.2, TR1.1 (CT), TR1.10 (CT), TR1.4 (CT), TR1.7 (CT)
- new net: D25.1 (K), Q8.1 (G), R37.2, R40.1
- new net: D24.2 (A), R40.2
- new net: C44.2, R42.1
- new net 3.3V_ENABLE: Module1.86 (+3.3v_(Output)), Q7.1 (G), U22.4 (EN)
- new net 5V_switched: J2.7 (Pin_7), J2.7 (Pin_7), Q6.3 (D), U13.3 (VI)
- new net D0N: J25.2, TR1.22 (MX1-)
- new net D0P: J25.1, TR1.23 (MX1+)
- new net D1N: J25.6, TR1.19 (MX2-)
- new net D1P: J25.3, TR1.20 (MX2+)
- new net D2N: J25.5, TR1.16 (MX3-)
- new net D2P: J25.4, TR1.17 (MX3+)
- new net D3N: J25.8, TR1.13 (MX4-)
- new net D3P: J25.7, TR1.14 (MX4+)
- new net LED_PWR: D1.2 (A), D2.2 (A), JP5.2 (B), R13.1, R15.1
- new net VC1: C46.1, D22.3, J15.1 (Pin_1), TR1.24 (CT)
- new net VC2: C45.1, D22.4, J15.3 (Pin_3), TR1.21 (CT)
- new net VC3: C44.1, D13.3, J15.5 (Pin_5), TR1.18 (CT)
- new net VC4: C42.1, D13.4, J15.7 (Pin_7), TR1.15 (CT)
- new net VOUTN: C39.2, D13.2 (-), D15.2 (A2), D22.2 (-), D25.2 (A), Q8.2 (S), R36.1, R37.1
- new net VOUTP: C26.1, C39.1, D13.1 (+), D15.1 (A1), D16.2 (A), D22.1 (+), D24.1 (K), R36.2
- new net ~{5V_EN}: J14.2 (Pin_2), SW4.2 (B), U3.5 (~{ON}/OFF)
- no-connect marks 35 -> 32
Other:
- note added: "(for devices that care, this one does not)"
- note added: "Gigabit POE"
- note added: "Jumper 1-2 and 3-4 For Mode A"
- note added: "Jumper 5-6 and 7-8 For Mode B"
- note added: "POE Out"
- note added: "POWER SUPPLY STUFF TBD"
- note added: "Power"
- note added: "Power over Ethernet in (optional)"
- note added: "SWITCH TO BETTER CAPACITORS"
- note added: "TODO: FIX SPI NAMING CIPO COPI controller/peripheral"
- note removed: "TODO: FIX SPI NAMING POSI PISO (primary/secondary)"
- moved on the sheet: C18, C19, C20, C27, C28, C5, D10, D11, D12, D17, D2, D3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
Changed lines of the file:
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@@
-(kicad_sch (version 20211123) (generator eeschema)
+(kicad_sch (version 20230121) (generator eeschema)
   (paper "A2")

Commit message: CM4 robot board almost done for Rev 3.5
Parts:
- removed C23: 10u, Capacitor_SMD:C_0805_2012Metric, symbol Device:C
- removed C27, C28: 47uF, Capacitor_SMD:CP_Elec_10x10, symbol Device:C_Polarized
- removed C34: 22pF, Capacitor_SMD:C_0603_1608Metric, symbol Device:C
- removed C35: 22uF 10v, Capacitor_SMD:C_0805_2012Metric, symbol Device:C
- removed C37: 22uF 6.3v, Capacitor_SMD:C_0603_1608Metric, symbol Device:C
- removed J17, J18, J19, J20: Conn_01x04, Connector_Molex:Molex_KK-254_AE-6410-04A_1x04_P2.54mm_Vertical, symbol Connector_Generic:Conn_01x04
- removed L3: 10uH, Inductor_SMD:L_Sunlord_SWPA5040S, symbol Device:L
- removed R14: R, symbol Device:R
- removed R33: 2.2k 1%, Resistor_SMD:R_0603_1608Metric, symbol Device:R
- removed U13: NCP1117-3.3_SOT223, Package_TO_SOT_SMD:SOT-223-3_TabPin2, symbol Regulator_Linear:NCP1117-3.3_SOT223
- removed U22: MT2492, Package_TO_SOT_SMD:SOT-23-6, symbol Regulator_Switching:AP3211K
- added C110: 10u, Capacitor_SMD:C_0805_2012Metric, symbol Device:C
- added C111: 4.7uF 100V, Capacitor_SMD:C_1210_3225Metric, symbol Device:C
- added C112: 100nF 100V, Capacitor_SMD:C_0805_2012Metric, symbol Device:C
- added C122: 1u, Capacitor_SMD:C_0603_1608Metric, symbol Device:C
- added C26 (x2): 47uF 63V solid, Capacitor_THT:CP_Radial_D8.0mm_P3.50mm, symbol Device:C_Polarized
- added C40: 0.1uF, Capacitor_SMD:C_0805_2012Metric, symbol Device:C
- added C41: 0.1uF, Capacitor_SMD:C_0603_1608Metric, symbol Device:C
- added D4: SMAJ51A, Diode_SMD:D_SMA, symbol Diode:SMF54A
- added J3 (x2): Encoder 1, parts:Ckmtw-W-2510S06P_1x06_P2.54mm_Vertical, symbol Connector_Generic:Conn_01x06
- added JP6 (x2), JP8, JP9: SolderJumper_2_Open, Jumper:SolderJumper-2_P1.3mm_Open_RoundedPad1.0x1.5mm, symbol Jumper:SolderJumper_2_Open
- added Q9: AO3401A, Package_TO_SOT_SMD:SOT-23, symbol Transistor_FET:AO3401A
- added R14, R17, R45, R47, R48, R49, R50: 10k, Resistor_SMD:R_0603_1608Metric, symbol MotorController:TAYLOR_RESISTOR
- added R46: 5.1k, Resistor_SMD:R_0603_1608Metric, symbol Device:R
- added R60, R61: 27, Resistor_SMD:R_0603_1608Metric, symbol Device:R
- added SW3: CONFIG SWITCH, Button_Switch_SMD:SW_DIP_SPSTx06_Slide_KingTek_DSHP06TS_W7.62mm_P1.27mm, symbol Switch:SW_DIP_x06
- added SW5: SW_SPDT, parts:CS12ANW03, symbol Switch:SW_SPDT
- added U21: FT231XS, Package_SO:SSOP-20_3.9x8.7mm_P0.635mm, symbol Interface_USB:FT231XS
- added U22, U27, U29, U30: SN74LVC1G07QDCKTQ1, Package_TO_SOT_SMD:SOT-353_SC-70-5, symbol acorn-motherboard:SN74LVC1G07QDCKTQ1
- added U24: ISL54222AIUZ, parts:ISL54222AIUZ, symbol 2021-10-22_05-57-19:ISL54222AIUZ
- added U27 (x2): USBLC6-2P6, Package_TO_SOT_SMD:SOT-666, symbol Power_Protection:USBLC6-2P6
- added U28: PCA9536D, Package_SO:SOIC-8_3.9x4.9mm_P1.27mm, symbol Interface_Expansion:PCA9536D
- added U32: TLV1117LV33DCYR, Package_TO_SOT_SMD:SOT-223-3_TabPin2, symbol Regulator_Linear:NCP1117-3.3_SOT223
- C36: value 22uF 6.3v -> 0.1uF; Field4 (none) -> Farnell; Field5 (none) -> 2611911; Field6 (none) -> RM EMK105 B7104KV-F; Field7 (none) -> TAIYO YUDEN EUROPE GMBH; Field8 (none) -> 110091611; LCSC C59461 -> C14663; Part Description (none) -> 0.1uF 10% 16V Ceramic Capacitor X7R 0402 (1005 Metric)
- C5: value 1000uF -> 1000uF 10v solid; footprint Capacitor_SMD:CP_Elec_10x10 -> Capacitor_THT:CP_Radial_D8.0mm_P3.50mm; LCSC C310843 -> C556213
- JP5: now in the parts list
- R16: LCSC C22949 -> C5126104
- R32: value R -> 2.2k 1%; footprint (none) -> Resistor_SMD:R_0603_1608Metric; Digikey (none) -> RMCF0805FT2K10CT-ND; LCSC (none) -> C4190; MPN (none) -> RMCF0805FT2K10
- R36: value 24.1k/1% -> 24k; LCSC (none) -> C2930261
- R77: value 82R -> 200R; LCSC C23255 -> C217868
Connections:
- net +3V3: now also D1.2 (A), JP5.2 (B), R13.1, R15.1, R32.2, C110.1, C40.1, C41.2, R17.1, R47.1, U21.15 (VCC), U21.3 (VCCIO), U22.5 (VCC), U24.10 (VDD), U32.2 (VO); no longer JP5.1 (A), U7.5 (OE)
- net +5V: now also JP8.1 (A), JP9.1 (A), Q9.2 (S), R14.1, R48.1, U27.2 (A), U27.5 (VBUS), U27.5 (VCC), U29.5 (VCC); no longer C11.1, C15.2, C16.2, D18.1 (VDD), D19.1 (VDD), D20.1 (VDD), D21.1 (VDD), D5.1 (VDD), D6.1 (VDD), D7.1 (VDD), J11.2 (Pin_2), J21.1 (Pin_1), JP3.3 (B), JP4.3 (B), U10.8 (VCC2), U11.8 (VCC2), U7.6 (VCCB)
- net 5V_switched: now also C11.1, D18.1 (VDD), D19.1 (VDD), D20.1 (VDD), D21.1 (VDD), D5.1 (VDD), D6.1 (VDD), D7.1 (VDD), J11.2 (Pin_2), J21.1 (Pin_1), JP3.3 (B), JP4.3 (B), U7.6 (VCCB), C122.1, JP9.2 (B), U32.3 (VI); no longer J2.7 (Pin_7), J2.7 (Pin_7)
- net ESTOP: now also U22.2 (A); no longer U15.2 (A)
- net GND: now also C36.2, R77.1, C110.2, C111.2, C112.2, C122.2, C26.2, C26.2, C40.2, C41.1, D4.2 (A2), J3.6 (Pin_6), J3.6 (Pin_6), R45.1, R49.2, R50.2, SW3.1, SW3.2, SW3.3, SW5.1 (A), U21.16 (GND), U21.6 (GND), U22.3 (GND), U24.5 (GND), U24.9 (*OE), U27.2 (GND), U27.2 (GND), U27.3 (GND), U28.4 (VSS), U29.2 (A), U29.3 (GND), U30.3 (GND), U32.1 (GND); no longer R77.2, U1.1 (/OE), U18.1 (/OE), U19.1 (/OE)
- net RX_GPIO15: now also U21.20 (TXD)
- net SCL6: now also U28.6 (SCL)
- net SDA6: now also U28.7 (SDA)
- net SERIALPWR1: now also J3.1 (Pin_1)
- net SERIALPWR2: now also J3.1 (Pin_1)
- net TX_GPIO14: now also U21.4 (RXD)
- net USBA_D_N: now also U27.1 (I/O1); no longer U5.8 (HSD1-)
- net USBA_D_P: now also U27.3 (I/O2); no longer U5.2 (HSD1+)
- net USBC_D_N: now also U27.4 (I/O2); no longer U5.7 (HSD2-)
- net USBC_D_P: now also U27.6 (I/O1); no longer U5.3 (HSD2+)
- net USBC_VBUS_IN: now also U27.5 (VBUS)
- net VMOT: now also C111.1, C112.1, C26.1, C26.1, D4.1 (A1)
- net at D2.1 (K): now also R77.2; no longer R77.1
- net at U14.23 (TXB): now also J3.4 (Pin_4)
- net at U14.24 (RXB): now also J3.5 (Pin_5)
- net at U14.3 (TXA): now also J3.2 (Pin_2)
- net at U14.4 (RXA): now also J3.3 (Pin_3)
- net at Q6.1 (G), Q7.3 (D): now also R14.2
- net ESTOP_SINK1: now reaches R32.1
- net ESTOP_SINK1: now also J2.1 (Pin_1), SW3.12, U22.1 (/OE)
- net 3.3V_PI_OUT: now reaches C36.1
- net 3.3V_PI_OUT: now also JP5.1 (A), Module1.86 (+3.3v_(Output)), U28.8 (VDD), U30.2 (A), U30.5 (VCC)
- net at U13.3 (TXA): now also J3.2 (Pin_2)
- net at U13.4 (RXA): now also J3.3 (Pin_3)
- net at U13.23 (TXB): now also J3.4 (Pin_4)
- net at U13.24 (RXB): now also J3.5 (Pin_5)
- net PI_n_LED_ACT: now reaches Module1.21 (PI_nLED_Activity), R10.1, TP1.1
- net EXTRA_GPIO: now reaches J14.1 (Pin_1)
- net EXTRA_GPIO: now also U28.5 (IO3)
- net 3.3V_ENABLE: no longer names the net of Q7.1 (G)
- net 3.3V_ENABLE: now also U30.4 (Y); no longer Module1.86 (+3.3v_(Output))
- net ESTOP_SINK renamed ESTOP_SINK2
- net ESTOP_SINK2: now also SW3.11; no longer J2.1 (Pin_1)
- removed net LED_PWR: D1.2 (A), D2.2 (A), JP5.2 (B), R13.1, R15.1
- new net: D2.2 (A), R46.1, U27.4 (Y)
- new net: Q9.1 (G), R48.2, U29.4 (Y)
- new net: U15.2 (A), U22.4 (Y)
- new net 3.3V_PI_CONTROL: R50.1, U28.2 (IO1), U30.1 (/OE)
- new net 5V_CAN_ENABLE: R49.1, U28.1 (IO0), U29.1 (/OE)
- new net 5V_switched_CAN: C15.2, C16.2, J2.7 (Pin_7), J2.7 (Pin_7), JP8.2 (B), Q9.3 (D), U10.8 (VCC2), U11.8 (VCC2)
- new net LED_EN_NONINVERTED: R45.2, R46.2, U7.5 (OE)
- new net SER_SELECT: R47.2, SW5.2 (B), U21.14 (~{RESET}), U24.1 (SEL), U28.3 (IO2)
- new net USBAP_D_N: U27.6 (I/O1), U5.8 (HSD1-)
- new net USBAP_D_P: U27.4 (I/O2), U5.2 (HSD1+)
- new net USBCP_D_N: JP6.2 (B), U24.6 (D-), U27.3 (I/O2)
- new net USBCP_D_P: JP6.2 (B), U24.4 (D+), U27.1 (I/O1)
- new net USB_DN: R61.2, U21.12 (USBDM)
- new net USB_DP: R60.2, U21.11 (USBDP)
- new net USB_SERIAL_D+: R60.1, U24.3 (HSD2+)
- new net USB_SERIAL_D-: R61.1, U24.7 (HSD2-)
- new net USB_SW_D+: JP6.1 (A), U24.2 (HSD1+), U5.3 (HSD2+)
- new net USB_SW_D-: JP6.1 (A), U24.8 (HSD1-), U5.7 (HSD2-)
- new net /LED_EN: R17.2, SW3.10, U1.1 (/OE), U18.1 (/OE), U19.1 (/OE), U27.1 (/OE)
Other:
- note added: "CAN BUS"
- note added: "CM4"
- note added: "Ethernet"
- note added: "GND selects HSD1 which is USB, otherwise Serial is selected"
- note added: "I/O"
- note added: "LEDs"
- note added: "Serial"
- note removed: "Gigabit POE"
- note removed: "POWER SUPPLY STUFF TBD"
- note removed: "SWITCH TO BETTER CAPACITORS"
- note removed: "TODO: FIX SPI NAMING CIPO COPI controller/peripheral"
- moved on the sheet: C10, C11, C12, C13, C14, C15, C16, C18, C19, C2, C20, C21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

Commit message: Updated Motherboard design files to latest version.
Parts:
- removed JP1, JP2: SolderJumper_2_Open, Jumper:SolderJumper-2_P1.3mm_Open_RoundedPad1.0x1.5mm, symbol Jumper:SolderJumper_2_Open
- removed SW3: CONFIG SWITCH, Button_Switch_SMD:SW_DIP_SPSTx06_Slide_KingTek_DSHP06TS_W7.62mm_P1.27mm, symbol Switch:SW_DIP_x06
- added C124: 1u, Capacitor_SMD:C_0603_1608Metric, symbol Device:C
- added C37, C49, C50: 0.1uF, Capacitor_SMD:C_0603_1608Metric, symbol Device:C
- added JP10: SolderJumper_2_Open, Jumper:SolderJumper-2_P1.3mm_Open_RoundedPad1.0x1.5mm, symbol Jumper:SolderJumper_2_Open
- added R51, R52: 5.1k, Resistor_SMD:R_0603_1608Metric, symbol Device:R
- added SW6: SW_DIP_x02, Button_Switch_SMD:SW_DIP_SPSTx02_Slide_KingTek_DSHP02TS_W7.62mm_P1.27mm, symbol Switch:SW_DIP_x02
- added SW7: CONFIG_SW, Button_Switch_SMD:SW_DIP_SPSTx04_Slide_KingTek_DSHP04TS_W7.62mm_P1.27mm, symbol Switch:SW_DIP_x04
- added TP2: TestPoint, TestPoint:TestPoint_Loop_D2.60mm_Drill1.6mm_Beaded, symbol Connector:TestPoint
- added U31: LSM6DS3, Package_LGA:LGA-14_3x2.5mm_P0.5mm_LayoutBorder3x4y, symbol Sensor_Motion:LSM6DS3
- added U32: LIS3MDL, Package_LGA:LGA-12_2x2mm_P0.5mm, symbol Sensor_Magnetic:LIS3MDL
- J22, J8, J9: now not fitted
- J3: value Encoder 1 -> ~
- JP5, JP8, JP9: now not fitted; now left out of the parts list
Connections:
- net +3V3: now also C124.1, C37.1, C50.1, JP10.1 (A), U31.12 (CS), U31.5 (VDDIO), U31.8 (VDD), U32.10 (~{CS}), U32.5 (Vdd), U32.6 (Vdd_IO)
- net CAN0_P: now also SW6.4
- net CAN1_P: now also SW6.3
- net ESTOP_SINK1: now also SW7.8
- net ESTOP_SINK2: now also SW7.7
- net GND: now also C124.2, C37.2, C49.2, C50.2, R51.1, R52.1, SW7.1, SW7.2, SW7.3, TP2.1, U31.2 (SDX), U31.3 (SCX), U31.6 (GND), U31.7 (GND), U32.12 (GND), U32.2 (GND), U32.3 (GND)
- net SCL6: now also U31.13 (SCL), U32.1 (SCL/SPC)
- net SDA6: now also U31.14 (SDA), U32.11 (SDA/SDI/SDO)
- net /LED_EN: now also SW7.6
- net at R35.2: now also SW6.2
- net at R34.2: now also SW6.1
- net 3.3V_PI_CONTROL renamed 3.3V_5V_PI_CONTROL
- net CAN_SCS0 renamed CAN_CS0
- net CAN_SCS1 renamed CAN_CS1
- net CAN_SI renamed CAN_COPI
- net CAN_SO renamed CAN_CIPO
- net SERIAL_SI renamed SERIAL_CIPO
- net SERIAL_SO renamed SERIAL_COPI
- new net: JP10.2 (B), R51.2, U31.1 (SDO/SA0)
- new net: C49.1, U32.4 (C1)
- new net: R52.2, U32.9 (SDO/SA1)
Other:
- note added: "Display"
- note added: "I2C address"
- note added: "LED Enable and E-Stop Config"
- note added: "Motion Sensing"
- note added: "Power Control"
- note added: "SPI Naming Note: COPI "Controller Out, Peripheral In" CIPO "Controller In, Peripheral Out" This is a slight deviation from OSHWA who recommend PICO/POCI, but those terms swap the order of the controller compared to previous terms, and I find MISO=CIPO easier to intuit than MISO=POCI."
- note added: "USB Serial"
- note added: "default to inputs with 100k internal pull-up resistor"
- note removed: "SPI naming note: I wanted to move away from master/slave naming but in doing so I used inconsistent and unclear conventions. -TLA TODO: Use "primary/secondary" and make everything PISO/POSI"
- moved on the sheet: C10, C11, C110, C111, C112, C12, C122, C13, C14, C15, C16, C18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
