File: cm4_robot_board/cm4-robot.kicad_sch (KiCad schematic)
At the start: 223 parts, among them J1 1747981-1, J10 Conn_01x04, J11 Conn_01x03, J12 Conn_01x04, J14 Conn_01x03, J15 Conn_02x04_Odd_Even, J2 CAN Interface, J21 Conn_01x03, J22 Conn_01x04, J23 Conn_01x01, J24 Conn_01x01, J25 RJ45, J3 USB_C_Receptacle_USB2.0, J4 Conn_01x04, J5 Conn_01x04, J6 Conn_01x04, J7 USB_A, J8 HIGHCURRENTPAD2, J9 HIGHCURRENTPAD2, Q1 Q_PMOS_GSD, Q2 Q_NMOS_GSD, Q3 Q_NMOS_GSD, Q4 Q_NMOS_GSD, Q5 Q_NMOS_GSD, Q6 AO3401A, Q7 AO3400A, Q8 Si2328DS, Q9 AO3401A, SW1 B3U-1000P, SW2 SW_SPDT, SW3 SW_SPDT, SW4 SW_SPDT, SW5 SW_SPDT, SW6 SW_DIP_x02, SW7 CONFIG_SW, U1 SN74LVC1G07QDCKTQ1, U10 isolator, U11 isolator, U12 TPS61040DBVR, U13 SC16IS752, U14 SC16IS752, U15 SN74LVC1G07QDCKTQ1, U16 CC56-12SEKWA, U17 ET6226M, U18 SN74LVC1G07QDCKTQ1, U19 SN74LVC1G07QDCKTQ1, U2 SN74LVC1G07QDCKTQ1, U21 FT231XS, U22 SN74LVC1G07QDCKTQ1, U23 TPD4E1U06DCKR, U24 ISL54222AIUZ, U27 SN74LVC1G07QDCKTQ1, U27 USBLC6-2P6, U28 PCA9536D, U29 SN74LVC1G07QDCKTQ1, U3 LM2576HVS-5, U30 SN74LVC1G07QDCKTQ1, U31 LSM6DS3, U32 LIS3MDL, U32 TLV1117LV33DCYR, U4 TPD4E1U06DCKR, U5 ISL54222AIUZ, U6 LTC4412xS6, U7 TXS0101DCKR, U8 MCP2515-xSO, U9 MCP2515-xSO, Y1 16MHz, Y2 16MHz, Y3 14.7456MHz, Y4 14.7456MHz

Commit message: Update motherboard, in progress not complete
Parts:
- removed J14: Conn_01x03, Connector_Molex:Molex_KK-254_AE-6410-03A_1x03_P2.54mm_Vertical, symbol Connector_Generic:Conn_01x03
- removed J15: Conn_02x04_Odd_Even, Connector_PinHeader_2.54mm:PinHeader_2x04_P2.54mm_Vertical, symbol Connector_Generic:Conn_02x04_Odd_Even
- removed J8, J9: HIGHCURRENTPAD2, parts:PAD_12GA_WIRE, symbol Connector_Generic:Conn_01x01
- removed R45: 10k, Resistor_SMD:R_0603_1608Metric, symbol MotorController:TAYLOR_RESISTOR
- added C52: 1u, Capacitor_SMD:C_0603_1608Metric, symbol Device:C
- added C53: 100n, Capacitor_SMD:C_0603_1608Metric, symbol Device:C
- added D27: 1N4148WS, Diode_SMD:D_SOD-323, symbol Device:D
- added D28, D29: LED_RED, LED_SMD:LED_0805_2012Metric, symbol Device:LED
- added D30: LED_Dual, parts:LED-SMD_4P-L2.0-W1.3-RD-TL, symbol Device:LED_Dual_KAKA
- added J8: Conn_01x02, Connector_Anderson:PowerPole_PP45_1336G1_1x2_Horizontal, symbol Connector_Generic:Conn_01x02
- added J9: POWER AND ESTOP, parts:BOOMELE-2510-5A _1x05_P2.54mm_Vertical, symbol Connector_Generic:Conn_01x05
- added JP1, JP11, JP12, JP13, JP14: SolderJumper_2_Open, Jumper:SolderJumper-2_P1.3mm_Open_RoundedPad1.0x1.5mm, symbol Jumper:SolderJumper_2_Open
- added JP2: SolderJumper_3_Open, Jumper:SolderJumper-3_P1.3mm_Open_RoundedPad1.0x1.5mm, symbol Jumper:SolderJumper_3_Open
- added Q10: Q_NMOS_GSD, Package_TO_SOT_SMD:SOT-23, symbol Device:Q_NMOS_GSD
- added R45, R59, R60: 220R, Resistor_SMD:R_0603_1608Metric, symbol Device:R
- added R53, R54: 50k 0.1%, Resistor_SMD:R_0603_1608Metric, symbol MotorController:TAYLOR_RESISTOR
- added R55: 5.1k 0.1%, Resistor_SMD:R_0603_1608Metric, symbol MotorController:TAYLOR_RESISTOR
- added R56, R57: 2.2k 1%, Resistor_SMD:R_0603_1608Metric, symbol Device:R
- added R58: 10k, Resistor_SMD:R_0603_1608Metric, symbol MotorController:TAYLOR_RESISTOR
- added U33: ADS1115IDGS, Package_SO:TSSOP-10_3x3mm_P0.5mm, symbol Analog_ADC:ADS1115IDGS
- added U34, U35, U36: SN74LVC1G07QDCKTQ1, Package_TO_SOT_SMD:SOT-353_SC-70-5, symbol acorn-motherboard:SN74LVC1G07QDCKTQ1
- R46: value 5.1k -> 220R; Digikey (none) -> A129741CT-ND; LCSC C23186 -> C22962
- R50: value 10k -> 100k; LCSC C25804 -> C14675
- U28: LCSC (none) -> C129522
Connections:
- net +3V3: now also C52.2, C53.1, D27.1 (K), JP2.1 (A), R56.2, R57.2, U33.8 (VDD), U34.2 (A), U34.5 (VCC), U35.5 (VCC), U36.5 (VCC); no longer C13.2, C14.2, C25.2, C26.2, C30.1, C31.1, D14.2 (A), D23.2 (A), D4.2 (A), R18.2, R19.2, R20.2, R21.2, R29.1, R30.1, R5.2, R6.2, U10.1 (VCC1), U11.1 (VCC1), U13.8 (VDD), U14.8 (VDD), U8.18 (VDD), U9.18 (VDD)
- net 3.3V_5V_PI_CONTROL: now also U30.2 (A); no longer R50.1, U30.1 (/OE)
- net 3.3V_PI_OUT: now also R29.1, R30.1, JP2.3 (B); no longer U30.2 (A)
- net ESTOP: now also U36.2 (A); no longer U22.2 (A)
- net ESTOP_OUT: now also U36.4 (Y); no longer D8.2 (A), U15.4 (Y)
- net EXTRA_GPIO: now also J9.3 (Pin_3)
- net GND: now also SW7.4, U22.2 (A), U30.1 (/OE), C52.1, C53.2, J8.2 (Pin_2), J9.2 (Pin_2), J9.5 (Pin_5), JP12.1 (A), JP14.1 (A), Q10.2 (S), R55.2, R58.1, U33.1 (ADDR), U33.3 (GND), U34.3 (GND), U35.3 (GND), U36.3 (GND); no longer D18.3 (VSS), D19.3 (VSS), D20.3 (VSS), D21.3 (VSS), D5.3 (VSS), D6.3 (VSS), D7.3 (VSS), J21.3 (Pin_3), R27.2, R50.2
- net LED_EN_NONINVERTED: no longer R46.2
- net SCL6: now also U33.10 (SCL)
- net SDA6: now also U33.9 (SDA)
- net VC1: now also JP11.2 (B)
- net VC2: now also JP12.2 (B)
- net VC3: now also JP13.2 (B)
- net VC4: now also JP14.2 (B)
- net VMOT: now also R50.1, J8.1 (Pin_1), JP1.2 (B), JP11.1 (A), JP13.1 (A), R53.1; no longer D16.1 (K)
- net /LED_EN: now also SW7.5, U34.1 (/OE); no longer SW7.6
- net ~{5V_EN}: now also R50.2, J9.4 (Pin_4)
- net at D2.2 (A), U27.4 (Y): no longer R46.1
- net at U15.2 (A), U22.4 (Y): now also R46.2
- new net: D29.1 (K), R46.1
- new net: D18.3 (VSS), D19.3 (VSS), D20.3 (VSS), D21.3 (VSS), D5.3 (VSS), D6.3 (VSS), D7.3 (VSS), J21.3 (Pin_3), Q10.3 (D)
- new net: R53.2, R54.1
- new net: D16.1 (K), JP1.1 (A)
- new net: D28.1 (K), R45.1
- new net: R45.2, U15.4 (Y), U35.2 (A)
- new net 3.3V_SEL: C13.2, C14.2, C25.2, C30.1, C31.1, JP2.2 (C), R18.2, R19.2, R20.2, R21.2, R5.2, R6.2, U10.1 (VCC1), U11.1 (VCC1), U13.8 (VDD), U8.18 (VDD), U9.18 (VDD)
- new net ESTOP_SINK_ALL: R27.2, R57.1, U35.4 (Y), U36.1 (/OE)
- new net ESTOP_SINK_LOCAL: J9.1 (Pin_1), R56.1, SW7.6, U35.1 (/OE)
- new net LED_3.3V_POWER_NONINV: D28.2 (A), D29.2 (A), D8.2 (A), Q10.1 (G), R58.2, U34.4 (Y)
- new net LED_3.3V_POWER_SW: D14.2 (A), D23.2 (A), D4.2 (A)
- new net SERIAL_CAN_PWR_3.3V: C26.2, U14.8 (VDD)
- new net VMEAS: D27.2 (A), R54.2, R55.1, U33.4 (AIN0)
Other:
- note added: "5V power"
- note added: "I2C Address 0x48"
- moved on the sheet: C111, C112, C18, C19, C20, C26, C39, D11, D16, D24, D25, D8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

Commit message: Update motherboard and add soft start pcb
Parts:
- removed D30: LED_Dual, parts:LED-SMD_4P-L2.0-W1.3-RD-TL, symbol Device:LED_Dual_KAKA
- removed J9: POWER AND ESTOP, parts:BOOMELE-2510-5A _1x05_P2.54mm_Vertical, symbol Connector_Generic:Conn_01x05
- added D30: LED_Dual_KKAA, parts:LED-ARRAY-SMD_4P-L1.9-W1.6-BL-CW, symbol cm4-robot:LED_Dual_KKAA
- added J14: Power Sw, Connector_Molex:Molex_KK-254_AE-6410-03A_1x03_P2.54mm_Vertical, symbol Connector_Generic:Conn_01x03
- added J9: ESTOP, Connector_Molex:Molex_KK-254_AE-6410-03A_1x03_P2.54mm_Vertical, symbol Connector_Generic:Conn_01x03
- J2: value CAN Interface -> M12A-08PFFR-SF7003; Name (none) -> CAN Interface
- J22: value Conn_01x04 -> DNP; now in the parts list
- R27, R45, R46, R59, R60: value 220R -> 130R; LCSC C22962 -> C22796
Connections:
- net 3.3V_SEL is gone; now on net SERIAL_CAN_PWR_3.3V: C13.2, C14.2, C25.2, C30.1, C31.1, JP2.2 (C), R18.2, R19.2, R20.2, R21.2, R5.2, R6.2, U10.1 (VCC1), U11.1 (VCC1), U13.8 (VDD), U8.18 (VDD), U9.18 (VDD)
- net LED_EN_NONINVERTED is gone; now on net LED_3.3V_POWER_NONINV: U7.5 (OE)
- net ESTOP_OUT: now also R60.2, D30.4 (A2)
- net ESTOP_SINK_LOCAL: now also J9.1 (Pin_1)
- net EXTRA_GPIO: now also J14.1 (Pin_1)
- net GND: now also J21.3 (Pin_3), R59.2, J14.3 (Pin_3), J9.3 (Pin_3)
- net LED_3.3V_POWER_NONINV: now also D30.3 (A1)
- net ~{5V_EN}: now also J14.2 (Pin_2)
- net at D18.3 (VSS), D19.3 (VSS), D20.3 (VSS)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: no longer J21.3 (Pin_3)
- net at R59.1: now also D30.1 (K1)
- net at R60.1: now also D30.2 (K2)
Other:
- note added: "3.3V_PI_OUT - always on 3.3v from pi, for GPIO expander +3.3V - switched 3.3v regulator, fed off 5v rail controlled by GPIO expander SERIAL_CAN_PWR_3.3V - jumper-selectable rail can feed from either of the two above. controls the serial and CAN chips, which have kernel modules that may or may not get unhappy if their chips reset We use an external 3.3v regulator because the Pi's onboard 3.3v regu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"
- note added: "Green"
- note added: "In an earlier rev it was discovered that this POE circuit works, but may connect the +V rail to workbench ground, causing issues when using USB cables. This circuit still works but will only be useful in certain circumstances, so it uses an optional jumper to connect. Long term, an isolated power converter should be added."
- note added: "Red"
