File: cm4_robot_board/cm4-robot.kicad_sch (KiCad schematic)
At the start: 248 parts, among them J1 1747981-1, J10 Conn_01x04, J11 Conn_01x03, J12 Conn_01x04, J14 Power Sw, J15 I2C OLED, J2 M12A-08PFFR-SF7003, J21 Conn_01x03, J22 DNP, J23 Conn_01x01, J24 Conn_01x01, J25 RJ45, J3 USB_C_Receptacle_USB2.0, J4 Conn_01x04, J5 Conn_01x04, J6 Conn_01x04, J7 USB_A, J8 Conn_01x02, J9 ESTOP, Q1 Q_PMOS_GSD, Q10 Q_NMOS_GSD, Q2 Q_NMOS_GSD, Q3 Q_NMOS_GSD, Q4 Q_NMOS_GSD, Q5 Q_NMOS_GSD, Q6 AO3401A, Q7 AO3400A, Q8 Si2328DS, Q9 AO3401A, SW1 B3U-1000P, SW2 SW_SPDT, SW3 SW_SPDT, SW4 SW_SPDT, SW5 SW_SPDT, SW6 SW_DIP_x02, SW7 CONFIG_SW, U1 SN74LVC1G07QDCKTQ1, U10 isolator, U11 isolator, U12 TPS61040DBVR, U13 SC16IS752, U14 SC16IS752, U15 SN74LVC1G07QDCKTQ1, U16 CC56-12SEKWA, U17 ET6226M, U18 SN74LVC1G07QDCKTQ1, U19 SN74LVC1G07QDCKTQ1, U2 SN74LVC1G07QDCKTQ1, U21 FT231XS, U22 SN74LVC1G07QDCKTQ1, U23 TPD4E1U06DCKR, U24 ISL54222AIUZ, U27 SN74LVC1G07QDCKTQ1, U27 USBLC6-2P6, U28 PCA9536D, U29 SN74LVC1G07QDCKTQ1, U3 LM2576HVS-5, U30 SN74LVC1G07QDCKTQ1, U31 LSM6DS3, U32 LIS3MDL, U32 TLV1117LV33DCYR, U33 ADS1115IDGS, U34 SN74LVC1G07QDCKTQ1, U35 SN74LVC1G07QDCKTQ1, U36 SN74LVC1G07QDCKTQ1, U4 TPD4E1U06DCKR, U5 ISL54222AIUZ, U6 LTC4412xS6, U7 TXS0101DCKR, U8 MCP2515-xSO, U9 MCP2515-xSO, Y1 16MHz, Y2 16MHz, Y3 14.7456MHz, Y4 14.7456MHz

Commit message: Motherboard: Add GPS port and other updates. Ready for review.
Parts:
- added J18: Serial Rear, Connector_PinSocket_2.54mm:PinSocket_2x05_P2.54mm_Vertical_SMD, symbol Connector_Generic:Conn_02x05_Odd_Even
- J10, J12, J4, J5, J6: LCSC C402777 -> C2982033
Connections:
- net GND: now also J18.1 (Pin_1)
- net SERIALPWR1: now also J18.2 (Pin_2)
- net TX4: now reaches J3.4 (Pin_4), U14.23 (TXB)
- net TX4: now also J18.8 (Pin_8)
- net RX4: now reaches J3.5 (Pin_5), U14.24 (RXB)
- net RX4: now also J18.10 (Pin_10)
- net TX3: now reaches J3.2 (Pin_2), U14.3 (TXA)
- net TX3: now also J18.4 (Pin_4)
- net RX3: now reaches J3.3 (Pin_3), U14.4 (RXA)
- net RX3: now also J18.6 (Pin_6)
- net TX2: now reaches J3.4 (Pin_4), U13.23 (TXB)
- net TX2: now also J18.7 (Pin_7)
- net RX2: now reaches J3.5 (Pin_5), U13.24 (RXB)
- net RX2: now also J18.9 (Pin_9)
- net TX1: now reaches J3.2 (Pin_2), U13.3 (TXA)
- net TX1: now also J18.3 (Pin_3)
- net RX1: now reaches J3.3 (Pin_3), U13.4 (RXA)
- net RX1: now also J18.5 (Pin_5)
Other:
- note added: "MAKE DIP SWITCH LARGER OR MOVE LEDS TO BIG SWITCH"
- note added: "MOUNT GPS ON BACK"
- moved on the sheet: C21, C22, C23, C24, C25, C26, J3, JP1, JP2, JP3, JP4, R18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
Changed lines of the file:
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@@
-(kicad_sch (version 20230121) (generator eeschema)
-  (paper "A1")
+(kicad_sch
+	(version 20231120)
+	(generator "eeschema")
+	(generator_version "8.0")
+	(paper "A1")

Commit message: remove extra schematic notes
Other:
- note removed: "MAKE DIP SWITCH LARGER OR MOVE LEDS TO BIG SWITCH"
- note removed: "MOUNT GPS ON BACK"

Commit message: update motherboard, add supercap_simple. ready for review
Parts:
- added J19: SBUS, parts:610108249221, symbol Connector_Generic:Conn_02x04_Odd_Even
- added JP15: SolderJumper_2_Open, Jumper:SolderJumper-2_P1.3mm_Open_RoundedPad1.0x1.5mm, symbol Jumper:SolderJumper_2_Open
- added R61, R62, R63: 10k, Resistor_SMD:R_0603_1608Metric, symbol MotorController:TAYLOR_RESISTOR
- added TP4, TP5, TP6: TestPoint, TestPoint:TestPoint_Pad_D2.0mm, symbol Connector:TestPoint
Connections:
- net +3V3: now also R61.1, R62.1, R63.1
- net 5V_switched: now also J19.5 (Pin_5), J19.6 (Pin_6)
- net ESTOP_SINK_ALL: now also R63.2
- net GND: now also J19.7 (Pin_7), J19.8 (Pin_8), JP15.2 (B); no longer R49.2
- net RC_SBUS: now also J19.3 (Pin_3), J19.4 (Pin_4)
- net at R46.2, U15.2 (A), U22.4 (Y): now also R61.2
- net at U33.5 (AIN1): now also TP4.1
- net at U33.6 (AIN2): now also TP5.1
- net at U33.7 (AIN3): now also TP6.1
- net at R45.2, U15.4 (Y), U35.2 (A): now also R62.2
- new net: JP15.1 (A), R49.2
Other:
- note added: "- July 10 2024 Expand E-stop circuit to provide indicator lights for each branch Add local motherboard branch of e-stop circuit Provide jumper to control whether external 5v over CAN is on or off at startup. Add extra SBUS connector to eliminate cabling. Add pullup resistor to power switch signals. Add I2C ADC for input voltage sensing"
- note added: "Changelog"
- note added: "In an earlier rev it was discovered that this POE circuit works, but some POE devices output inverted power, so this power supply should be isolated. However under certain use cases POE can still be used, so a jumper was inserted until it can be properly fixed."
- note removed: "In an earlier rev it was discovered that this POE circuit works, but may connect the +V rail to workbench ground, causing issues when using USB cables. This circuit still works but will only be useful in certain circumstances, so it uses an optional jumper to connect. Long term, an isolated power converter should be added."
- moved on the sheet: C36, C52, D28, D29, D30, D8, J11, JP5, JP9, Q7, Q9, R12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

Commit message: Resolve most of the schematic ERC errors.
Parts:
- C53: value 100n -> 0.1u; LCSC (none) -> C14663
- D15: LCSC (none) -> C7466458
- R37: LCSC (none) -> C3016651
Connections:
- no-connect marks 32 -> 146
Other:
- moved on the sheet: C10, C11, C110, C111, C12, C122, C124, C13, C16, C18, C19, C20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

Commit message: Update with most design review feedback. Needs final checkout.
Parts:
- added D31: Diode Dual Common Cathode 80v maximum reverse vol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, Package_TO_SOT_SMD:SOT-323_SC-70, symbol Device:D_Dual_CommonCathode_AAK
- added F2: Polyfuse, Fuse:Fuse_1206_3216Metric, symbol Device:Polyfuse
- added R64: 10K, Resistor_SMD:R_0603_1608Metric, symbol MotorController:TAYLOR_RESISTOR
- C10, C4, C7, C8: value 18p -> 18pF 50V; MPN (none) -> CL10C180JB8NNNC; Manufacturer (none) -> Samsung Electro-Mechanics
- C11, C12, C13, C14, C15, C16, C25, C26, C30, C31, C36, C37, C41, C47, C49, C50, C6, C9: value 0.1uF -> 0.1uF 50V; MPN (none) -> CC0603KRX7R9BB104; Manufacturer (none) -> YAGEO
- C110, C20: value 10u -> 10uF 25V; MPN (none) -> CL21A106KAYNNNE; Manufacturer (none) -> Samsung Electro-Mechanics
- C111: MPN (none) -> C3225X7S2A475KT000N; Manufacturer (none) -> TDK
- C112: MPN (none) -> CL21B104KCFNNNE; Manufacturer (none) -> Samsung Electro-Mechanics
- C122, C124, C52: value 1u -> 1uF 50V; MPN (none) -> CL10A105KB8NNNC; Manufacturer (none) -> Samsung Electro-Mechanics
- C18: value 4.7uF -> 4.7uF 25V; MPN (none) -> CL10A475KA8NQNC; Manufacturer (none) -> Samsung Electro-Mechanics
- C19: value 22pF -> 22pF 50V; MPN (none) -> CL10C220JB8NNNC; Manufacturer (none) -> Samsung Electro-Mechanics
- C2, C3: value 10uF -> 10uF 25V; MPN CC0805ZKY5V6BB106 -> CL21A106KAYNNNE; Manufacturer (none) -> Samsung Electro-Mechanics
- C20: value 1uF -> 1uF 25V; MPN (none) -> 0603B105K250NT; Manufacturer (none) -> FH (Guangdong Fenghua Advanced Tech)
- C21, C22, C23, C24: value 22p -> 22pF 50V; MPN (none) -> CL10C220JB8NNNC; Manufacturer (none) -> Samsung Electro-Mechanics
- C26: MPN (none) -> 4700630811R00; Manufacturer (none) -> NJCON
- C29: MPN (none) -> RVT1A471M0607; Manufacturer (none) -> ROQANG
- C33, C38: MPN (none) -> GRM32ER61C476KE15L; Manufacturer (none) -> Murata Electronics
- C39: value 0.1uF -> 0.1uF 100V; MPN (none) -> CL21B104KCFNNNE; Manufacturer (none) -> Samsung Electro-Mechanics
- C40: value 0.1uF -> 0.1uF 50V; MPN (none) -> 0805B104K500NT
- C42, C44, C45, C46: MPN (none) -> CC0603KRX7R0BB223; Manufacturer (none) -> YAGEO
- C43: MPN (none) -> 1206B102K202NT; Manufacturer (none) -> FH (Guangdong Fenghua Advanced Tech)
- C5: MPN (none) -> SPT1AM102F12OR; Manufacturer (none) -> Yunxing
- C53: value 0.1u -> 0.1uF 50V; MPN (none) -> CC0603KRX7R9BB104; Manufacturer (none) -> YAGEO
- D1, D17, D23: MPN SML-LX1206SOC-TR -> TC0805YF01-1CSA; Manufacturer (none) -> TCWIN
- D10, D9: MPN CDSOT23-SM712 -> SM712; Manufacturer (none) -> TECH PUBLIC
- D11: MPN (none) -> MBR0530; Manufacturer (none) -> Jiangsu Changjing Electronics Technology Co., Ltd.
- D12, D14: MPN (none) -> KT-0805G; Manufacturer (none) -> Hubei KENTO Elec
- D13, D22: MPN (none) -> ABS210; Manufacturer (none) -> Guangdong Hottech
- D15: MPN (none) -> SMAJ60A; Manufacturer (none) -> HXY MOSFET
- D16: MPN (none) -> M7; Manufacturer (none) -> MDD(Microdiode Semiconductor)
- D18, D19, D20, D21, D5, D6, D7: MPN (none) -> WS2812B-B/T; Manufacturer (none) -> Worldsemi
- D2, D28, D29, D8: MPN LTST-C150KRKT -> NCD0805R1; Manufacturer (none) -> Foshan NationStar Optoelectronics
- D24: MPN (none) -> MMSZ5255B_R1_00001; Manufacturer (none) -> PANJIT International
- D25: MPN (none) -> BZT52C15S; Manufacturer (none) -> Jiangsu Changjing Electronics Technology Co., Ltd.
- D27: MPN (none) -> 1N4148WS; Manufacturer (none) -> Jiangsu Changjing Electronics Technology Co., Ltd.
- D3: MPN (none) -> SS510C; Manufacturer (none) -> Shandong Jingdao Microelectronics
- D30: MPN (none) -> 19-22/R6GHC-A32/2T; Manufacturer (none) -> Everlight Elec
- D4: Manufacturer (none) -> TCWIN
- D4: MPN (none) -> SMAJ51A; Manufacturer (none) -> TWGMC
- F1: MPN (none) -> nSMD010; Manufacturer (none) -> TECHFUSE
- J1: MPN 1747981-1 -> HDMI-01; Manufacturer (none) -> HCTL
- J10, J12, J4, J5, J6: MPN 0022232041 -> HC-2510-4A; Manufacturer (none) -> HCTL
- J11, J14, J21, J9: MPN (none) -> 744-81-03TW10; Manufacturer (none) -> PINREX
- J15: MPN (none) -> 2.54-1*4P; Manufacturer (none) -> BOOMELE(Boom Precision Elec); Note (none) -> 128x64 Pixel SH1106 I2C OLED widely available on Amazon or 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
- J18: MPN (none) -> 2.54-2*5P; Manufacturer (none) -> BOOMELE(Boom Precision Elec)
- J23, J24, Module1: MPN (none) -> DF40HC(3.0)-100DS-0.4V(51); Manufacturer (none) -> HRS(Hirose)
- J25: MPN (none) -> R-RJ45R08P-B000; Manufacturer (none) -> Ckmtw(Shenzhen Cankemeng)
- J3: MPN (none) -> HC-2510-6A; Manufacturer (none) -> HCTL
- J3: MPN (none) -> TYPEC-304J-BCP16; Manufacturer (none) -> XUNPU
- J7: MPN UE27AC54100 -> 902-131A1011D10100; Manufacturer (none) -> Jing Extension of the Electronic Co.
- L1: MPN (none) -> YPRH1508-101M; Manufacturer (none) -> YJYCOIN
- L2: MPN (none) -> NLCV32T-100K-PF; Manufacturer (none) -> TDK
- Q1: MPN (none) -> AO3401A; Manufacturer (none) -> UMW(Youtai Semiconductor Co., Ltd.)
- Q10, Q2, Q3, Q4, Q5: MPN (none) -> NX7002AK,215; Manufacturer (none) -> Nexperia
- Q6, Q9: MPN (none) -> AO3401A; Manufacturer (none) -> BORN
- Q7: MPN (none) -> AO3400A; Manufacturer (none) -> UMW(Youtai Semiconductor Co., Ltd.)
- Q8: Manufacturer (none) -> Diodes Incorporated
- R1, R10: MPN (none) -> 0603WAF1001T5E; Manufacturer (none) -> UNI-ROYAL(Uniroyal Elec)
- R11, R32, R4, R56, R57, R9: MPN RMCF0805FT2K10 -> 0603WAF2201T5E; Manufacturer (none) -> UNI-ROYAL(Uniroyal Elec)
- R12, R14, R17, R23, R28, R29, R30, R47, R48, R49, R5, R58, R6, R61, R62, R63: value 10k -> 10K; MPN (none) -> 0603WAF1002T5E; Manufacturer (none) -> UNI-ROYAL(Uniroyal Elec)
- R13: MPN (none) -> 0603WAF270JT5E; Manufacturer (none) -> UNI-ROYAL(Uniroyal Elec)
- R15: MPN (none) -> 0603WAF560JT5E; Manufacturer (none) -> UNI-ROYAL(Uniroyal Elec)
- R16: MPN (none) -> FRC0603F2053TS; Manufacturer (none) -> FOJAN
- R18, R20: MPN (none) -> AR03BTCX1002; Manufacturer (none) -> Viking Tech
- R19, R21: MPN (none) -> RC0603FR-071KL; Manufacturer (none) -> YAGEO
- R2, R3: MPN (none) -> 0603WAF4700T5E; Manufacturer (none) -> UNI-ROYAL(Uniroyal Elec)
- R22, R24, R25, R26: MPN (none) -> RC0603FR-07100RL; Manufacturer (none) -> YAGEO
- R27, R45, R46, R59, R60: MPN (none) -> 0603WAF1300T5E; Manufacturer (none) -> UNI-ROYAL(Uniroyal Elec)
- R34, R35: MPN (none) -> 0603WAF1200T5E; Manufacturer (none) -> UNI-ROYAL(Uniroyal Elec)
- R36: MPN (none) -> FRC0805J240TSD; Manufacturer (none) -> FOJAN
- R37: MPN (none) -> SCR0805F249K; Manufacturer (none) -> VO
- R40: MPN (none) -> 0805W8F5102T5E; Manufacturer (none) -> UNI-ROYAL(Uniroyal Elec)
- R41, R42, R43, R44: MPN (none) -> PTFR0603B75R0N9; Manufacturer (none) -> RESI
- R50: MPN (none) -> RC0603FR-07100KL; Manufacturer (none) -> YAGEO
- R51, R52, R7, R8: MPN (none) -> 0603WAF5101T5E; Manufacturer (none) -> UNI-ROYAL(Uniroyal Elec)
- R53, R54: MPN (none) -> AR03BTC5002A; Manufacturer (none) -> Viking Tech
- R55: MPN (none) -> RT0603BRD075K1L; Manufacturer (none) -> YAGEO
- R60, R61: value 27 -> 27R; MPN (none) -> 0603WAF270JT5E; Manufacturer (none) -> UNI-ROYAL(Uniroyal Elec)
- R77: MPN (none) -> ARG03FTC2000; Manufacturer (none) -> Viking Tech
- SW1: MPN (none) -> TS-1101-C-W; Manufacturer (none) -> XKB Connection
- SW2, SW3, SW4, SW5: MPN (none) -> SS-12D10L5; Manufacturer (none) -> XKB Connection
- SW6: MPN (none) -> DSHP02TSGET; Manufacturer (none) -> DongGuan KINGTEK Industrial Co.,LTD
- SW7: MPN (none) -> DSHP04TSGET; Manufacturer (none) -> DongGuan KINGTEK Industrial Co.,LTD
- TR1: MPN (none) -> G2401CG; Manufacturer (none) -> Dongguan Mentech Optical & Magnetic
- U1, U15, U18, U19, U2, U22, U27, U29, U30, U34, U35, U36: MPN TC7SH34FU,LJ(CT -> U74LVC1G125G-AL5-R; Manufacturer (none) -> UTC(Unisonic Tech)
- U10, U11: MPN (none) -> CA-IS3050G; Manufacturer (none) -> Chipanalog
- U13, U14: MPN (none) -> SC16IS752IPW,128; Manufacturer (none) -> NXP Semicon
- U16: MPN (none) -> FJ5461AH; Manufacturer (none) -> Shenzhen Zhihao Elec
- U17: MPN (none) -> ET6226M; Manufacturer (none) -> UMW(Youtai Semiconductor Co., Ltd.)
- U21: MPN (none) -> FT231XS-R; Manufacturer (none) -> FTDI
- U23, U4: Manufacturer (none) -> Texas Instruments
- U24, U5: MPN ISL54222AIUZ -> MSUSB30; Manufacturer (none) -> Hangzhou Ruimeng Tech
- U27: MPN (none) -> USBLC6-2P6; Manufacturer (none) -> TECH PUBLIC
- U28: MPN (none) -> PCA9536D; Manufacturer (none) -> NXP Semicon
- U3: MPN (none) -> LM2576HVS-5.0/TR; Manufacturer (none) -> HGSEMI
- U31: MPN (none) -> LSM6DSOWTR; Manufacturer (none) -> STMicroelectronics
- U32: MPN (none) -> LIS3MDLTR; Manufacturer (none) -> STMicroelectronics
- U32: MPN (none) -> TLV1117LV33DCYR; Manufacturer (none) -> Texas Instruments
- U33: MPN (none) -> ADS1115IDGSR; Manufacturer (none) -> Texas Instruments
- U6: MPN (none) -> LTC4412ES6#TRPBF; Manufacturer (none) -> Analog Devices
- U7: MPN (none) -> TXS0101DCKR; Manufacturer (none) -> Texas Instruments
- U8, U9: MPN (none) -> MCP2515T-I/SO; Manufacturer (none) -> Microchip Tech
- Y1, Y2: MPN (none) -> TXM16M0004322DBCDO00T; Manufacturer (none) -> Yajingxin
- Y3, Y4: MPN (none) -> SX3B14.7456F2010F30; Manufacturer (none) -> Shenzhen SCTF Elec
Connections:
- net +3V3: now also U21.13 (3V3OUT)
- net +5V: now also F2.2; no longer J7.1 (VBUS), U27.5 (VBUS)
- net GND: no longer U6.3 (CTL)
- net USBC_VBUS_IN: now also R64.2
- net ~{5V_EN}: now also D31.3 (K); no longer R50.2, U3.5 (~{ON}/OFF)
- new net 5V_FUSED: F2.1, J7.1 (VBUS), U27.5 (VBUS)
- new net ~{VBUS_5V_ENA}: D31.2 (A), R64.1, U6.3 (CTL)
- new net ~{VIN_5V_EN}: D31.1 (A), R50.2, U3.5 (~{ON}/OFF)
- no-connect marks 146 -> 145
Other:
- moved on the sheet: D4, J12, J7, J8, JP15, JP5, JP6, JP8, JP9, Q1, Q2, Q3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

Commit message: Updated board files for July 2024 order. Added supercap_simple.
Parts:
- added C54: 0.1uF 50V, Capacitor_SMD:C_0603_1608Metric, symbol Device:C
- added TP7: TestPoint, TestPoint:TestPoint_Pad_D2.0mm, symbol Connector:TestPoint
- C112: value 100nF 100V -> 0.1uF 100V
- C33, C38: value 47uF 16V -> 47uF 16V
- D1, D17, D23: Digikey 67-1696-1-ND -> (none); LCSC C5137318 -> C965814; MPN TC0805YF01-1CSA -> XL-2012UYC; Manufacturer TCWIN -> XINGLIGHT
- D15: LCSC C7466458 -> C707480; Manufacturer HXY MOSFET -> FTR
- D4: Digikey 160-1404-1-ND -> (none); LCSC C5137315 -> C965815; MPN LTST-C150KGKT -> XL-2012UGC; Manufacturer TCWIN -> XINGLIGHT
- J2: value M12A-08PFFR-SF7003 -> CAN Interface A; Name CAN Interface -> CAN Interface A
- J2: value M12A-08PFFR-SF7003 -> CAN Interface B; Name CAN Interface -> CAN Interface B
- J7: value USB_A -> USB HOSTING OUT
- R17: LCSC C177951 -> C403036
- R18, R20: Digikey 311-10.0KCRCT-ND -> (none); LCSC C319939 -> C25804; MPN AR03BTCX1002 -> (none); Manufacturer Viking Tech -> (none)
- TP1: LCSC C238130 -> C238131
Connections:
- net +5V: now also C54.1
- net GND: now also C54.2, TP7.1
Other:
- moved on the sheet: C33, C38, C5, L1
